Commit message: update the meshes parts of the xacro

File: xacro/quadruped.urdf.xacro (robot description, xacro)
@@ -27,5 +27,5 @@
         <geometry>
           <!-- <cylinder length="${upper_leg_length}" radius="${upper_leg_radius}"/> -->
-          <mesh filename="package://quadruped/urdf/cylinder.obj" scale="${upper_leg_radius} ${upper_leg_radius} ${upper_leg_length}"/>
+          <mesh filename="package://quadruped/meshes/cylinder.obj" scale="${upper_leg_radius} ${upper_leg_radius} ${upper_leg_length}"/>
         </geometry>
         <material name="grey">
@@ -65,5 +65,5 @@
         <geometry>
           <!-- <cylinder length="${upper_leg_length}" radius="${upper_leg_radius}"/> -->
-          <mesh filename="package://quadruped/urdf/cylinder.obj" scale="${upper_leg_radius} ${upper_leg_radius} ${upper_leg_length}"/>
+          <mesh filename="package://quadruped/meshes/cylinder.obj" scale="${upper_leg_radius} ${upper_leg_radius} ${upper_leg_length}"/>
         </geometry>
         <material name="grey">
@@ -100,5 +100,5 @@
         <geometry>
           <!-- <sphere radius="${upper_leg_radius}"/> -->
-          <mesh filename="package://quadruped/urdf/sphere.obj" scale="${upper_leg_radius} ${upper_leg_radius} ${upper_leg_radius}"/>
+          <mesh filename="package://quadruped/meshes/sphere.obj" scale="${upper_leg_radius} ${upper_leg_radius} ${upper_leg_radius}"/>
         </geometry>
         <material name="red">
@@ -130,5 +130,5 @@
         <origin rpy="0 0 0" xyz="0 0 0"/>
         <geometry>
-          <mesh filename="package://quadruped/urdf/cube.obj" scale="${base_w} ${base_l} ${base_h}"/>
+          <mesh filename="package://quadruped/meshes/cube.obj" scale="${base_w} ${base_l} ${base_h}"/>
             <!-- <box size="${base_w} ${base_l} ${base_h}"/> -->
         </geometry>

Commit message: update the xacro file so that it works in 14.04: 1**2 is corrected to 1*1

File: xacro/quadruped.urdf.xacro (robot description, xacro)
@@ -1,4 +1,4 @@
 <?xml version="1.0" ?>
-<robot name="quadroped"
+<robot name="quadruped"
   xmlns:controller="http://playerstage.sourceforge.net/gazebo/xmlschema/#controller"
   xmlns:interface="http://playerstage.sourceforge.net/gazebo/xmlschema/#interface"
@@ -125,5 +125,9 @@
         <origin rpy="0 0 0" xyz="0 0 0"/>
         <mass value="${base_m}"/>
-        <inertia ixx="${1./12. * base_m * (base_h**2 + base_l**2)}" ixy="0" ixz="0" iyy="${1./12. * base_m * (base_h**2 + base_w**2)}" iyz="0" izz="${1./12. * base_m * (base_w**2 + base_l**2)}"/>
+        <inertia ixx="${1./12. * base_m * (base_h*base_h + base_l*base_l)}"
+                 ixy="0" ixz="0"
+                 iyy="${1./12. * base_m * (base_h*base_h + base_w*base_w)}"
+                 iyz="0" izz="${1./12. * base_m * (base_w*base_w + base_l*base_l)}"
+        />
     </inertial>
     <visual>
@@ -131,5 +135,4 @@
         <geometry>
           <mesh filename="package://quadruped/meshes/cube.obj" scale="${base_w} ${base_l} ${base_h}"/>
-            <!-- <box size="${base_w} ${base_l} ${base_h}"/> -->
         </geometry>
         <material name="white">
@@ -145,7 +148,8 @@
   </link>
   <!-- <xacro:leg prefix="FL" rx="${0.}" ry="${0.}"/> -->
+<!--
   <xacro:leg prefix="FL" rx="${-0.5*base_w}" ry="${0.5*base_l}"/>
   <xacro:leg prefix="FR" rx="${+0.5*base_w}" ry="${0.5*base_l}"/>
   <xacro:leg prefix="HL" rx="${-0.5*base_w}" ry="${-0.5*base_l}"/>
-  <xacro:leg prefix="HR" rx="${+0.5*base_w}" ry="${-0.5*base_l}"/>
+  <xacro:leg prefix="HR" rx="${+0.5*base_w}" ry="${-0.5*base_l}"/> -->
 </robot>

Commit message: Fix direction of joint rotation axis.

File: xacro/quadruped.urdf.xacro (robot description, xacro)
@@ -18,5 +18,5 @@
       <child link="${prefix}_upperleg"/>
       <limit effort="1000" lower="-10" upper="10" velocity="1000"/>
-      <axis xyz="1 0 0"/>
+      <axis xyz="-1 0 0"/>
       <origin rpy="0 0 0" xyz="${rx} ${ry} 0"/>
       <dynamics damping="0.0" friction="0.0"/>
@@ -52,5 +52,5 @@
       <child link="${prefix}_shank"/>
       <limit effort="1000" velocity="10000"/>
-      <axis xyz="1 0 0"/>
+      <axis xyz="-1 0 0"/>
       <origin rpy="0 0 0" xyz="0 0 ${-upper_leg_length}"/>
       <dynamics damping="0.0" friction="0.0"/>

Commit message: Adjust quadruped xacro/urdf to new convetion: X axis is into the front

File: xacro/quadruped.urdf.xacro (robot description, xacro)
@@ -18,5 +18,5 @@
       <child link="${prefix}_upperleg"/>
       <limit effort="1000" lower="-10" upper="10" velocity="1000"/>
-      <axis xyz="-1 0 0"/>
+      <axis xyz="0 1 0"/>
       <origin rpy="0 0 0" xyz="${rx} ${ry} 0"/>
       <dynamics damping="0.0" friction="0.0"/>
@@ -46,5 +46,5 @@
           iyy="0.000469609"
           izz="1e-6"/>
-    </inertial>
+      </inertial>
     </link>
     <joint name="${prefix}_KFE" type="revolute">
@@ -52,5 +52,5 @@
       <child link="${prefix}_shank"/>
       <limit effort="1000" velocity="10000"/>
-      <axis xyz="-1 0 0"/>
+      <axis xyz="0 1 0"/>
       <origin rpy="0 0 0" xyz="0 0 ${-upper_leg_length}"/>
       <dynamics damping="0.0" friction="0.0"/>
@@ -125,8 +125,8 @@
         <origin rpy="0 0 0" xyz="0 0 0"/>
         <mass value="${base_m}"/>
-        <inertia ixx="${1./12. * base_m * (base_h*base_h + base_l*base_l)}"
-                 ixy="0" ixz="0"
-                 iyy="${1./12. * base_m * (base_h*base_h + base_w*base_w)}"
-                 iyz="0" izz="${1./12. * base_m * (base_w*base_w + base_l*base_l)}"
+        <inertia ixx="${1./12. * base_m * (base_h*base_h + base_w*base_w)}"
+                 iyy="${1./12. * base_m * (base_h*base_h + base_l*base_l)}"
+                 izz="${1./12. * base_m * (base_w*base_w + base_l*base_l)}"
+                 ixy="0" ixz="0" iyz="0"
         />
     </inertial>
@@ -134,5 +134,5 @@
         <origin rpy="0 0 0" xyz="0 0 0"/>
         <geometry>
-          <mesh filename="package://quadruped/meshes/cube.obj" scale="${base_w} ${base_l} ${base_h}"/>
+          <mesh filename="package://quadruped/meshes/cube.obj" scale="${base_l} ${base_w} ${base_h}"/>
         </geometry>
         <material name="white">
@@ -143,12 +143,12 @@
         <origin rpy="0 0 0" xyz="0 0 0"/>
         <geometry>
-            <box size="${base_w} ${base_l} ${base_h}"/>
+            <box size="${base_l} ${base_w} ${base_h}"/>
         </geometry>
     </collision>
   </link>
   <!-- <xacro:leg prefix="FL" rx="${0.}" ry="${0.}"/> -->
-  <xacro:leg prefix="FL" rx="${-0.5*base_w}" ry="${0.5*base_l}"/>
-  <xacro:leg prefix="FR" rx="${+0.5*base_w}" ry="${0.5*base_l}"/>
-  <xacro:leg prefix="HL" rx="${-0.5*base_w}" ry="${-0.5*base_l}"/>
-  <xacro:leg prefix="HR" rx="${+0.5*base_w}" ry="${-0.5*base_l}"/>
+  <xacro:leg prefix="FL" ry="${+0.5*base_w}" rx="${0.5*base_l}"/>
+  <xacro:leg prefix="FR" ry="${-0.5*base_w}" rx="${0.5*base_l}"/>
+  <xacro:leg prefix="HL" ry="${+0.5*base_w}" rx="${-0.5*base_l}"/>
+  <xacro:leg prefix="HR" ry="${-0.5*base_w}" rx="${-0.5*base_l}"/>
 </robot>

Commit message: update th place of teh meshes so that rviz and pybullet can load the urdf file and the meshes

File: xacro/quadruped.urdf.xacro (robot description, xacro)
@@ -27,5 +27,5 @@
         <geometry>
           <!-- <cylinder length="${upper_leg_length}" radius="${upper_leg_radius}"/> -->
-          <mesh filename="package://quadruped/meshes/cylinder.obj" scale="${upper_leg_radius} ${upper_leg_radius} ${upper_leg_length}"/>
+          <mesh filename="package://robot_properties_quadruped/meshes/cylinder.obj" scale="${upper_leg_radius} ${upper_leg_radius} ${upper_leg_length}"/>
         </geometry>
         <material name="grey">
@@ -65,5 +65,5 @@
         <geometry>
           <!-- <cylinder length="${upper_leg_length}" radius="${upper_leg_radius}"/> -->
-          <mesh filename="package://quadruped/meshes/cylinder.obj" scale="${upper_leg_radius} ${upper_leg_radius} ${upper_leg_length}"/>
+          <mesh filename="package://robot_properties_quadruped/meshes/cylinder.obj" scale="${upper_leg_radius} ${upper_leg_radius} ${upper_leg_length}"/>
         </geometry>
         <material name="grey">
@@ -100,5 +100,5 @@
         <geometry>
           <!-- <sphere radius="${upper_leg_radius}"/> -->
-          <mesh filename="package://quadruped/meshes/sphere.obj" scale="${upper_leg_radius} ${upper_leg_radius} ${upper_leg_radius}"/>
+          <mesh filename="package://robot_properties_quadruped/meshes/sphere.obj" scale="${upper_leg_radius} ${upper_leg_radius} ${upper_leg_radius}"/>
         </geometry>
         <material name="red">
@@ -134,5 +134,5 @@
         <origin rpy="0 0 0" xyz="0 0 0"/>
         <geometry>
-          <mesh filename="package://quadruped/meshes/cube.obj" scale="${base_l} ${base_w} ${base_h}"/>
+          <mesh filename="package://robot_properties_quadruped/meshes/cube.obj" scale="${base_l} ${base_w} ${base_h}"/>
         </geometry>
         <material name="white">
