Commit message: add back the material for the obj and switch to stl meshes for the display in gepetto viewer.

File: xacro/solo.urdf.xacro (robot description, xacro)
@@ -8,5 +8,5 @@
   <xacro:property name="color" value="0.8 0.8 0.8" />
   <xacro:property name="opacity" value="1.0" />
-  <xacro:property name="mesh_ext" value="obj" />
+  <xacro:property name="mesh_ext" value="stl" />
   <!-- This file is based on: https://atlas.is.localnet/confluence/display/AMDW/Quadruped+URDF+Files -->
   <link name="base_link">
