Commit message: Adjust the mass to match current hardware

File: xacro/solo12.urdf.xacro (robot description, xacro)
@@ -14,5 +14,5 @@
     <inertial>
         <origin xyz="0 0 0" rpy="0 0 0" />
-        <mass value="1.63315091"/>
+        <mass value="1.36115091"/>
         <!-- The base is extremely symmetrical. -->
         <inertia ixx="0.00578574" ixy="0.0" ixz="0.0"

Commit message: Solo12: Reduce total mass to 2.5 kg matching latest robot version

File: xacro/solo12.urdf.xacro (robot description, xacro)
@@ -14,5 +14,5 @@
     <inertial>
         <origin xyz="0 0 0" rpy="0 0 0" />
-        <mass value="1.36115091"/>
+        <mass value="1.16115091"/>
         <!-- The base is extremely symmetrical. -->
         <inertia ixx="0.00578574" ixy="0.0" ixz="0.0"
