Commit message: update the inertia and the meshes of the quadruped.urdf.xacro

File: xacro/leg.xacro (robot description, xacro)
@@ -12,4 +12,9 @@
   <xacro:property name="KFE_2_contact_y" value="${0 * 0.001}" />
   <xacro:property name="KFE_2_contact_z" value="${(160.00 + 0.5*27) * 0.001}" />
+  <!-- Inertia computation -->
+  <xacro:property name="upper_leg_length" value="0.16" />
+  <xacro:property name="upper_leg_radius" value="0.025" />
+  <xacro:property name="upper_leg_mass" value="0.162" />
+  <xacro:property name="lower_leg_mass" value="0.021" />
   <!-- This macro has for purpose to define a left leg -->
   <xacro:macro name="leg" params="prefix is_front is_right mesh_ext
@@ -46,10 +51,9 @@
       <inertial>
         <origin rpy="0 0 0" xyz="0 0 -0.0793"/>
-        <mass value="1.0"/>
+        <mass value="${upper_leg_mass}"/>
         <inertia ixy="0.0" ixz="0.0" iyz="0.0"
           ixx="0.000469609"
           iyy="0.000469609"
-          izz="1e-6"
-        />
+          izz="1e-6"/>
       </inertial>
       <!-- UPPER LEG LINK VISUAL -->
@@ -115,12 +119,12 @@
     <link name="${prefix}_lower_leg">
       <!-- LOWER LEG LINK INERTIAL -->
-      <inertial>
+       <inertial>
         <origin rpy="0 0 0" xyz="0 0 -0.0756"/>
-        <mass value="1.0"/>
+        <mass value="${lower_leg_mass + 0.01}"/>
         <inertia ixy="0.0" ixz="0.0" iyz="0.0"
           ixx="0.000087575"
           iyy="0.000087575"
           izz="1e-6"/>
-      </inertial>
+     </inertial>
       <!-- LOWER LEG LINK VISUAL -->
       <visual>

File: xacro/quadruped.urdf.xacro (robot description, xacro)
@@ -5,121 +5,15 @@
   xmlns:sensor="http://playerstage.sourceforge.net/gazebo/xmlschema/#sensor"
   xmlns:xacro="http://playerstage.sourceforge.net/gazebo/xmlschema/#interface">
+  <xacro:property name="color_name" value="grey" />
+  <xacro:property name="color" value="0.8 0.8 0.8" />
+  <xacro:property name="opacity" value="1.0" />
+  <xacro:property name="mesh_ext" value="obj" />
+  <!-- Inertia computation -->
   <xacro:property name="base_w" value=".2" />
   <xacro:property name="base_l" value=".4" />
   <xacro:property name="base_h" value=".05" />
   <xacro:property name="base_m" value="2.0" />
-  <xacro:property name="upper_leg_length" value="0.16" />
-  <xacro:property name="upper_leg_radius" value="0.025" />
-  <xacro:property name="upper_leg_mass" value="0.162" />
-  <xacro:property name="lower_leg_mass" value="0.021" />
-  <xacro:macro name="leg" params="prefix rx ry">
-    <joint name="${prefix}_HFE" type="revolute">
-      <parent link="base_link"/>
-      <child link="${prefix}_upperleg"/>
-      <limit effort="1000" lower="-10" upper="10" velocity="1000"/>
-      <axis xyz="0 1 0"/>
-      <origin rpy="0 0 0" xyz="${rx} ${ry} 0"/>
-      <dynamics damping="0.0" friction="0.0"/>
-    </joint>
-    <link name="${prefix}_upperleg">
-      <visual>
-        <origin rpy="0 0 0" xyz="0 0 ${-.5*upper_leg_length}"/>
-        <geometry>
-          <!-- <cylinder length="${upper_leg_length}" radius="${upper_leg_radius}"/> -->
-          <mesh filename="package://robot_properties_quadruped/meshes/cylinder.obj" scale="${upper_leg_radius} ${upper_leg_radius} ${upper_leg_length}"/>
-        </geometry>
-        <material name="grey">
-          <color rgba=".4 .4 .4 .1"/>
-        </material>
-      </visual>
-      <collision>
-        <origin rpy="0 0 0" xyz="0 0 ${-.5*upper_leg_length}"/>
-        <geometry>
-          <cylinder length="${upper_leg_length}" radius="${upper_leg_radius}"/>
-        </geometry>
-      </collision>
-      <inertial>
-        <origin rpy="0 0 0" xyz="0 0 -0.0793"/>
-        <mass value="${upper_leg_mass}"/>
-        <inertia ixy="0.0" ixz="0.0" iyz="0.0"
-          ixx="0.000469609"
-          iyy="0.000469609"
-          izz="1e-6"/>
-      </inertial>
-    </link>
-    <joint name="${prefix}_KFE" type="revolute">
-      <parent link="${prefix}_upperleg"/>
-      <child link="${prefix}_shank"/>
-      <limit effort="1000" velocity="10000"/>
-      <axis xyz="0 1 0"/>
-      <origin rpy="0 0 0" xyz="0 0 ${-upper_leg_length}"/>
-      <dynamics damping="0.0" friction="0.0"/>
-    </joint>
-    <link name="${prefix}_shank">
-      <contact>
-          <lateral_friction value="1.0"/>
-          <restitution value="0.5"/>
-      </contact>
-      <visual>
-        <origin rpy="0 0 0" xyz="0 0 ${-.5*upper_leg_length}"/>
-        <geometry>
-          <!-- <cylinder length="${upper_leg_length}" radius="${upper_leg_radius}"/> -->
-          <mesh filename="package://robot_properties_quadruped/meshes/cylinder.obj" scale="${upper_leg_radius} ${upper_leg_radius} ${upper_leg_length}"/>
-        </geometry>
-        <material name="grey">
-          <color rgba=".4 .4 .4 .1"/>
-        </material>
-      </visual>
-      <collision>
-        <origin rpy="0 0 0" xyz="0 0 ${-.5*upper_leg_length}"/>
-        <geometry>
-          <cylinder length="${upper_leg_length}" radius="${upper_leg_radius}"/>
-        </geometry>
-      </collision>
-      <inertial>
-        <origin rpy="0 0 0" xyz="0 0 -0.0756"/>
-        <mass value="${lower_leg_mass}"/>
-        <inertia ixy="0.0" ixz="0.0" iyz="0.0"
-          ixx="0.000087575"
-          iyy="0.000087575"
-          izz="1e-6"/>
-    </inertial>
-    </link>
-    <joint name="${prefix}_END" type="fixed">
-      <parent link="${prefix}_shank"/>
-      <child link="${prefix}_contact"/>
-      <origin rpy="0 0 0" xyz="0 0 ${-upper_leg_length}"/>
-    </joint>
-    <link name="${prefix}_contact">
-      <contact>
-          <lateral_friction value="1.0"/>
-          <restitution value="0.5"/>
-      </contact>
-      <visual>
-        <origin rpy="0 0 0" xyz="0 0 0"/>
-        <geometry>
-          <!-- <sphere radius="${upper_leg_radius}"/> -->
-          <mesh filename="package://robot_properties_quadruped/meshes/sphere.obj" scale="${upper_leg_radius} ${upper_leg_radius} ${upper_leg_radius}"/>
-        </geometry>
-        <material name="red">
-          <color rgba="1. 0. 0. 1."/>
-        </material>
-      </visual>
-      <collision>
-        <origin rpy="0 0 0" xyz="0 0 0"/>
-        <geometry>
-          <sphere radius="${upper_leg_radius}"/>
-        </geometry>
-      </collision>
-      <inertial>
-        <mass value="0.01"/>
-        <inertia ixy="0.0" ixz="0.0" iyz="0.0"
-          ixx="0."
-          iyy="0."
-          izz="0."/>
-    </inertial>
-    </link>
-  </xacro:macro>
   <link name="base_link">
+    <!-- BASE LINK INERTIAL -->
     <inertial>
         <origin rpy="0 0 0" xyz="0 0 0"/>
@@ -131,24 +25,62 @@
         />
     </inertial>
+    <!-- BASE LINK VISUAL -->
     <visual>
         <origin rpy="0 0 0" xyz="0 0 0"/>
         <geometry>
-          <mesh filename="package://robot_properties_quadruped/meshes/cube.obj" scale="${base_l} ${base_w} ${base_h}"/>
+          <mesh filename="package://robot_properties_quadruped/meshes/${mesh_ext}/quadruped_body.${mesh_ext}"/>
         </geometry>
-        <material name="white">
-            <color rgba="1 1 1 1"/>
+        <material name="${color_name}">
+            <color rgba="${color} ${opacity}"/>
         </material>
     </visual>
+    <!-- BASE LINK COLLISION -->
     <collision>
         <origin rpy="0 0 0" xyz="0 0 0"/>
         <geometry>
-            <box size="${base_l} ${base_w} ${base_h}"/>
+          <mesh filename="package://robot_properties_quadruped/meshes/${mesh_ext}/quadruped_body.${mesh_ext}"/>
         </geometry>
+        <material name="${color_name}">
+            <color rgba="${color} ${opacity}"/>
+        </material>
     </collision>
-  </link>
-  <!-- <xacro:leg prefix="FL" rx="${0.}" ry="${0.}"/> -->
-  <xacro:leg prefix="FL" ry="${+0.5*base_w}" rx="${0.5*base_l}"/>
-  <xacro:leg prefix="FR" ry="${-0.5*base_w}" rx="${0.5*base_l}"/>
-  <xacro:leg prefix="HL" ry="${+0.5*base_w}" rx="${-0.5*base_l}"/>
-  <xacro:leg prefix="HR" ry="${-0.5*base_w}" rx="${-0.5*base_l}"/>
+  </link> <!-- END BASE LINK -->
+  <!-- Include the legs -->
+  <xacro:include filename="leg.xacro"/>
+  <!-- Include the front left leg -->
+  <xacro:leg
+      prefix="FL"
+      is_front="true"
+      is_right="false"
+      mesh_ext="${mesh_ext}"
+      color_name="${color_name}"
+      color="${color}"
+      opacity="${opacity}"/>
+  <!-- Include the front right leg -->
+  <xacro:leg
+      prefix="FR"
+      is_front="true"
+      is_right="true"
+      mesh_ext="${mesh_ext}"
+      color_name="${color_name}"
+      color="${color}"
+      opacity="${opacity}"/>
+  <!-- Include the hind left leg -->
+  <xacro:leg
+      prefix="HL"
+      is_front="false"
+      is_right="false"
+      mesh_ext="${mesh_ext}"
+      color_name="${color_name}"
+      color="${color}"
+      opacity="${opacity}"/>
+  <!-- Include the hind right leg -->
+  <xacro:leg
+      prefix="HR"
+      is_front="false"
+      is_right="true"
+      mesh_ext="${mesh_ext}"
+      color_name="${color_name}"
+      color="${color}"
+      opacity="${opacity}"/>
 </robot>

File: xacro/quadruped_visual.urdf.xacro (robot description, xacro)
@@ -9,12 +9,17 @@
   <xacro:property name="opacity" value="1.0" />
   <xacro:property name="mesh_ext" value="obj" />
+  <!-- Inertia computation -->
+  <xacro:property name="base_w" value=".2" />
+  <xacro:property name="base_l" value=".4" />
+  <xacro:property name="base_h" value=".05" />
+  <xacro:property name="base_m" value="2.0" />
   <link name="base_link">
     <!-- BASE LINK INERTIAL -->
     <inertial>
         <origin rpy="0 0 0" xyz="0 0 0"/>
-        <mass value="2.0"/>
-        <inertia ixx="1.0"
-                 iyy="1.0"
-                 izz="1.0"
+        <mass value="${base_m}"/>
+        <inertia ixx="${1./12. * base_m * (base_h*base_h + base_w*base_w)}"
+                 iyy="${1./12. * base_m * (base_h*base_h + base_l*base_l)}"
+                 izz="${1./12. * base_m * (base_w*base_w + base_l*base_l)}"
                  ixy="0" ixz="0" iyz="0"
         />

Commit message: update the legg to have a foot link with no inertia

File: xacro/leg.xacro (robot description, xacro)
@@ -23,5 +23,5 @@
     <joint name="${prefix}_HFE" type="revolute">
       <parent link="base_link"/>
-      <child link="${prefix}_upper_leg"/>
+      <child link="${prefix}_UPPER_LEG"/>
       <limit effort="1000" lower="-10" upper="10" velocity="1000"/>
       <!-- joints rotates around the y-axis -->
@@ -47,5 +47,5 @@
       <dynamics damping="0.0" friction="0.0"/>
     </joint>
-    <link name="${prefix}_upper_leg">
+    <link name="${prefix}_UPPER_LEG">
       <!-- UPPER LEG LINK INERTIAL -->
       <inertial>
@@ -90,8 +90,6 @@
     <!-- KFE: Joint between the upper leg and the lower leg -->
     <joint name="${prefix}_KFE" type="revolute">
-      <parent link="${prefix}_upper_leg"/>
-      <child link="${prefix}_lower_leg"/>
-      <parent link="base_link"/>
-      <child link="${prefix}_upper_leg"/>
+      <parent link="${prefix}_UPPER_LEG"/>
+      <child link="${prefix}_LOWER_LEG"/>
       <limit effort="1000" lower="-10" upper="10" velocity="1000"/>
       <!-- joints rotates around the y-axis -->
@@ -117,7 +115,7 @@
       <dynamics damping="0.0" friction="0.0"/>
     </joint>
-    <link name="${prefix}_lower_leg">
+    <link name="${prefix}_LOWER_LEG">
       <!-- LOWER LEG LINK INERTIAL -->
-       <inertial>
+      <inertial>
         <origin rpy="0 0 0" xyz="0 0 -0.0756"/>
         <mass value="${lower_leg_mass + 0.01}"/>
@@ -158,4 +156,17 @@
       </collision>
     </link> <!-- END LOWER LEG LINK -->
+    <!-- KFE: Joint between the upper leg and the lower leg -->
+    <joint name="${prefix}_ANKLE" type="fixed">
+      <parent link="${prefix}_LOWER_LEG"/>
+      <child link="${prefix}_FOOT"/>
+      <!-- Joint placement -->
+      <origin xyz="0 0 ${-HFE_2_KFE_z}" rpy="0 0 0" />
+      <!-- Limits (usefull?) -->
+      <limit effort="1000" lower="-10" upper="10" velocity="1000"/>
+      <!-- pybullet simulation parameters -->
+      <dynamics damping="0.0" friction="0.0"/>
+    </joint>
+    <link name="${prefix}_FOOT">
+    </link>
   </xacro:macro>
 </robot>

Commit message: add the stl files with the foot for the collision checking in bullet

File: xacro/leg.xacro (robot description, xacro)
@@ -62,8 +62,8 @@
         <geometry>
           <xacro:unless value="${is_right}">
-            <mesh filename="package://robot_properties_quadruped/meshes/${mesh_ext}/quadruped_upper_leg_left_side.${mesh_ext}"/>
+            <mesh filename="package://robot_properties_quadruped/meshes/${mesh_ext}/stl_with_foot/quadruped_upper_leg_left_side.${mesh_ext}"/>
           </xacro:unless>
           <xacro:if value="${is_right}">
-            <mesh filename="package://robot_properties_quadruped/meshes/${mesh_ext}/quadruped_upper_leg_right_side.${mesh_ext}"/>
+            <mesh filename="package://robot_properties_quadruped/meshes/${mesh_ext}/stl_with_foot/quadruped_upper_leg_right_side.${mesh_ext}"/>
           </xacro:if>
         </geometry>
@@ -77,8 +77,8 @@
         <geometry>
           <xacro:unless value="${is_right}">
-            <mesh filename="package://robot_properties_quadruped/meshes/${mesh_ext}/quadruped_upper_leg_left_side.${mesh_ext}"/>
+            <mesh filename="package://robot_properties_quadruped/meshes/${mesh_ext}/stl_with_foot/quadruped_upper_leg_left_side.${mesh_ext}"/>
           </xacro:unless>
           <xacro:if value="${is_right}">
-            <mesh filename="package://robot_properties_quadruped/meshes/${mesh_ext}/quadruped_upper_leg_right_side.${mesh_ext}"/>
+            <mesh filename="package://robot_properties_quadruped/meshes/${mesh_ext}/stl_with_foot/quadruped_upper_leg_right_side.${mesh_ext}"/>
           </xacro:if>
         </geometry>
@@ -130,8 +130,8 @@
         <geometry>
           <xacro:unless value="${is_right}">
-            <mesh filename="package://robot_properties_quadruped/meshes/${mesh_ext}/quadruped_lower_leg_left_side.${mesh_ext}"/>
+            <mesh filename="package://robot_properties_quadruped/meshes/${mesh_ext}/stl_with_foot/quadruped_lower_leg_left_side.${mesh_ext}"/>
           </xacro:unless>
           <xacro:if value="${is_right}">
-            <mesh filename="package://robot_properties_quadruped/meshes/${mesh_ext}/quadruped_lower_leg_right_side.${mesh_ext}"/>
+            <mesh filename="package://robot_properties_quadruped/meshes/${mesh_ext}/stl_with_foot/quadruped_lower_leg_right_side.${mesh_ext}"/>
           </xacro:if>
         </geometry>
@@ -145,8 +145,8 @@
         <geometry>
           <xacro:unless value="${is_right}">
-            <mesh filename="package://robot_properties_quadruped/meshes/${mesh_ext}/quadruped_lower_leg_left_side.${mesh_ext}"/>
+            <mesh filename="package://robot_properties_quadruped/meshes/${mesh_ext}/stl_with_foot/quadruped_lower_leg_left_side.${mesh_ext}"/>
           </xacro:unless>
           <xacro:if value="${is_right}">
-            <mesh filename="package://robot_properties_quadruped/meshes/${mesh_ext}/quadruped_lower_leg_right_side.${mesh_ext}"/>
+            <mesh filename="package://robot_properties_quadruped/meshes/${mesh_ext}/stl_with_foot/quadruped_lower_leg_right_side.${mesh_ext}"/>
           </xacro:if>
         </geometry>

File: xacro/quadruped.urdf.xacro (robot description, xacro)
@@ -29,5 +29,5 @@
         <origin rpy="0 0 0" xyz="0 0 0"/>
         <geometry>
-          <mesh filename="package://robot_properties_quadruped/meshes/${mesh_ext}/quadruped_body.${mesh_ext}"/>
+          <mesh filename="package://robot_properties_quadruped/meshes/${mesh_ext}/stl_with_foot/quadruped_body.${mesh_ext}"/>
         </geometry>
         <material name="${color_name}">
@@ -39,5 +39,5 @@
         <origin rpy="0 0 0" xyz="0 0 0"/>
         <geometry>
-          <mesh filename="package://robot_properties_quadruped/meshes/${mesh_ext}/quadruped_body.${mesh_ext}"/>
+          <mesh filename="package://robot_properties_quadruped/meshes/${mesh_ext}/stl_with_foot/quadruped_body.${mesh_ext}"/>
         </geometry>
         <material name="${color_name}">

Commit message: update the urdf with a foot and with the bullet paramters. Behavior seems fine

File: xacro/leg.xacro (robot description, xacro)
@@ -62,8 +62,8 @@
         <geometry>
           <xacro:unless value="${is_right}">
-            <mesh filename="package://robot_properties_quadruped/meshes/${mesh_ext}/stl_with_foot/quadruped_upper_leg_left_side.${mesh_ext}"/>
-          </xacro:unless>
-          <xacro:if value="${is_right}">
-            <mesh filename="package://robot_properties_quadruped/meshes/${mesh_ext}/stl_with_foot/quadruped_upper_leg_right_side.${mesh_ext}"/>
+            <mesh filename="package://robot_properties_quadruped/meshes/${mesh_ext}/with_foot/quadruped_upper_leg_left_side.${mesh_ext}"/>
+          </xacro:unless>
+          <xacro:if value="${is_right}">
+            <mesh filename="package://robot_properties_quadruped/meshes/${mesh_ext}/with_foot/quadruped_upper_leg_right_side.${mesh_ext}"/>
           </xacro:if>
         </geometry>
@@ -77,8 +77,8 @@
         <geometry>
           <xacro:unless value="${is_right}">
-            <mesh filename="package://robot_properties_quadruped/meshes/${mesh_ext}/stl_with_foot/quadruped_upper_leg_left_side.${mesh_ext}"/>
-          </xacro:unless>
-          <xacro:if value="${is_right}">
-            <mesh filename="package://robot_properties_quadruped/meshes/${mesh_ext}/stl_with_foot/quadruped_upper_leg_right_side.${mesh_ext}"/>
+            <mesh filename="package://robot_properties_quadruped/meshes/${mesh_ext}/with_foot/quadruped_upper_leg_left_side.${mesh_ext}"/>
+          </xacro:unless>
+          <xacro:if value="${is_right}">
+            <mesh filename="package://robot_properties_quadruped/meshes/${mesh_ext}/with_foot/quadruped_upper_leg_right_side.${mesh_ext}"/>
           </xacro:if>
         </geometry>
@@ -87,4 +87,9 @@
         </material>
       </collision>
+      <!-- Bullet specific paramters -->
+      <contact>
+        <lateral_friction value="1.0"/>
+        <restitution value="0.5"/>
+      </contact>
     </link> <!-- END UPPER LEG LINK -->
     <!-- KFE: Joint between the upper leg and the lower leg -->
@@ -119,5 +124,5 @@
       <inertial>
         <origin rpy="0 0 0" xyz="0 0 -0.0756"/>
-        <mass value="${lower_leg_mass + 0.01}"/>
+        <mass value="${lower_leg_mass}"/>
         <inertia ixy="0.0" ixz="0.0" iyz="0.0"
           ixx="0.000087575"
@@ -130,8 +135,8 @@
         <geometry>
           <xacro:unless value="${is_right}">
-            <mesh filename="package://robot_properties_quadruped/meshes/${mesh_ext}/stl_with_foot/quadruped_lower_leg_left_side.${mesh_ext}"/>
-          </xacro:unless>
-          <xacro:if value="${is_right}">
-            <mesh filename="package://robot_properties_quadruped/meshes/${mesh_ext}/stl_with_foot/quadruped_lower_leg_right_side.${mesh_ext}"/>
+            <mesh filename="package://robot_properties_quadruped/meshes/${mesh_ext}/with_foot/quadruped_lower_leg_left_side.${mesh_ext}"/>
+          </xacro:unless>
+          <xacro:if value="${is_right}">
+            <mesh filename="package://robot_properties_quadruped/meshes/${mesh_ext}/with_foot/quadruped_lower_leg_right_side.${mesh_ext}"/>
           </xacro:if>
         </geometry>
@@ -145,8 +150,8 @@
         <geometry>
           <xacro:unless value="${is_right}">
-            <mesh filename="package://robot_properties_quadruped/meshes/${mesh_ext}/stl_with_foot/quadruped_lower_leg_left_side.${mesh_ext}"/>
-          </xacro:unless>
-          <xacro:if value="${is_right}">
-            <mesh filename="package://robot_properties_quadruped/meshes/${mesh_ext}/stl_with_foot/quadruped_lower_leg_right_side.${mesh_ext}"/>
+            <mesh filename="package://robot_properties_quadruped/meshes/${mesh_ext}/with_foot/quadruped_lower_leg_left_side.${mesh_ext}"/>
+          </xacro:unless>
+          <xacro:if value="${is_right}">
+            <mesh filename="package://robot_properties_quadruped/meshes/${mesh_ext}/with_foot/quadruped_lower_leg_right_side.${mesh_ext}"/>
           </xacro:if>
         </geometry>
@@ -155,4 +160,9 @@
         </material>
       </collision>
+      <!-- Bullet specific paramters -->
+      <contact>
+        <lateral_friction value="1.0"/>
+        <restitution value="0.5"/>
+      </contact>
     </link> <!-- END LOWER LEG LINK -->
     <!-- KFE: Joint between the upper leg and the lower leg -->
@@ -168,5 +178,39 @@
     </joint>
     <link name="${prefix}_FOOT">
-    </link>
+      <!-- FOOT INERTIAL -->
+      <inertial>
+        <origin rpy="0 0 0" xyz="0 0 0"/>
+        <mass value="0.01"/>
+        <inertia ixy="0.0" ixz="0.0" iyz="0.0"
+          ixx="0.0"
+          iyy="0.0"
+          izz="0.0"/>
+     </inertial>
+      <!-- FOOT VISUAL -->
+      <visual>
+        <origin rpy="0 0 0" xyz="0 0 0"/>
+        <geometry>
+          <mesh filename="package://robot_properties_quadruped/meshes/${mesh_ext}/with_foot/quadruped_foot.${mesh_ext}"/>
+        </geometry>
+        <material name="${color_name}">
+            <color rgba="${color} ${opacity}"/>
+        </material>
+      </visual>
+      <!-- FOOT COLLISION -->
+      <collision>
+        <origin rpy="0 0 0" xyz="0 0 0"/>
+        <geometry>
+            <mesh filename="package://robot_properties_quadruped/meshes/${mesh_ext}/with_foot/quadruped_foot.${mesh_ext}"/>
+        </geometry>
+        <material name="${color_name}">
+            <color rgba="${color} ${opacity}"/>
+        </material>
+      </collision>
+      <!-- Bullet specific paramters -->
+      <contact>
+        <lateral_friction value="1.0"/>
+        <restitution value="0.5"/>
+      </contact>
+    </link> <!-- END LOWER LEG LINK -->
   </xacro:macro>
 </robot>

File: xacro/quadruped.urdf.xacro (robot description, xacro)
@@ -29,5 +29,5 @@
         <origin rpy="0 0 0" xyz="0 0 0"/>
         <geometry>
-          <mesh filename="package://robot_properties_quadruped/meshes/${mesh_ext}/stl_with_foot/quadruped_body.${mesh_ext}"/>
+          <mesh filename="package://robot_properties_quadruped/meshes/${mesh_ext}/with_foot/quadruped_body.${mesh_ext}"/>
         </geometry>
         <material name="${color_name}">
@@ -39,5 +39,5 @@
         <origin rpy="0 0 0" xyz="0 0 0"/>
         <geometry>
-          <mesh filename="package://robot_properties_quadruped/meshes/${mesh_ext}/stl_with_foot/quadruped_body.${mesh_ext}"/>
+          <mesh filename="package://robot_properties_quadruped/meshes/${mesh_ext}/with_foot/quadruped_body.${mesh_ext}"/>
         </geometry>
         <material name="${color_name}">
@@ -45,4 +45,9 @@
         </material>
     </collision>
+    <!-- Bullet specific paramters -->
+    <contact>
+      <lateral_friction value="1.0"/>
+      <restitution value="0.5"/>
+    </contact>
   </link> <!-- END BASE LINK -->
   <!-- Include the legs -->
