Commit message: update the urdf

File: xacro/leg.xacro (robot description, xacro)
@@ -1,4 +1,4 @@
 <?xml version="1.0"?>
-<robot xmlns:xacro="http://playerstage.sourceforge.net/gazebo/xmlschema/#interface" name="athena">
+<robot xmlns:xacro="http://playerstage.sourceforge.net/gazebo/xmlschema/#interface" name="solo">
   <!-- See TODO: add the wiki link here -->
   <!-- These are absoulte distance value, the sign are decided below -->
@@ -12,9 +12,4 @@
   <xacro:property name="KFE_2_contact_y" value="${0 * 0.001}" />
   <xacro:property name="KFE_2_contact_z" value="${(160.00 + 0.5*27) * 0.001}" />
-  <!-- Inertia computation -->
-  <xacro:property name="upper_leg_length" value="0.16" />
-  <xacro:property name="upper_leg_radius" value="0.025" />
-  <xacro:property name="upper_leg_mass" value="0.162" />
-  <xacro:property name="lower_leg_mass" value="0.021" />
   <!-- This macro has for purpose to define a left leg -->
   <xacro:macro name="leg" params="prefix is_front is_right mesh_ext
@@ -49,15 +44,27 @@
     <link name="${prefix}_UPPER_LEG">
       <!-- UPPER LEG LINK INERTIAL -->
-      <inertial>
-        <origin rpy="0 0 0" xyz="0 0 -0.0793"/>
-        <mass value="${upper_leg_mass}"/>
-        <inertia ixy="0.0" ixz="0.0" iyz="0.0"
-          ixx="0.000469609"
-          iyy="0.000469609"
-          izz="1e-6"/>
-      </inertial>
+      <xacro:unless value="${is_right}">
+        <!-- Left upper leg inertia -->
+        <inertial>
+        <origin xyz="0.00001377 0.01935853 -0.07870700" rpy="0 0 0" />
+        <mass value="0.14853845"/>
+        <inertia ixx="0.00041107" ixy="0.0"         ixz="0.0"
+                                   iyy="0.00041193" iyz="0.00004671"
+                                                    izz="0.00003024"/>
+        </inertial>
+      </xacro:unless>
+      <xacro:if value="${is_right}">
+        <!-- Right upper leg inertia -->
+        <inertial>
+        <origin xyz="-0.00001377 -0.01935853 -0.07870700" rpy="0 0 0" />
+        <mass value="0.14853845"/>
+        <inertia ixx="0.00041107" ixy="0.0"         ixz="0.0"
+                                   iyy="0.00041193" iyz="-0.00004671"
+                                                    izz="0.00003024"/>
+        </inertial>
+      </xacro:if>
       <!-- UPPER LEG LINK VISUAL -->
       <visual>
-        <origin rpy="0 0 0" xyz="0 0 0"/>
+        <origin xyz="0 0 0" rpy="0 0 0" />
         <geometry>
           <xacro:unless value="${is_right}">
@@ -74,5 +81,5 @@
       <!-- UPPER LEG LINK COLLISION -->
       <collision>
-        <origin rpy="0 0 0" xyz="0 0 0"/>
+        <origin xyz="0 0 0" rpy="0 0 0" />
         <geometry>
           <xacro:unless value="${is_right}">
@@ -122,15 +129,27 @@
     <link name="${prefix}_LOWER_LEG">
       <!-- LOWER LEG LINK INERTIAL -->
-      <inertial>
-        <origin rpy="0 0 0" xyz="0 0 -0.0756"/>
-        <mass value="${lower_leg_mass}"/>
-        <inertia ixy="0.0" ixz="0.0" iyz="0.0"
-          ixx="0.000087575"
-          iyy="0.000087575"
-          izz="1e-6"/>
-     </inertial>
+      <xacro:unless value="${is_right}">
+        <!-- Left lower leg inertia -->
+        <inertial>
+        <origin xyz="0.0 0.00787644 -0.08928215" rpy="0 0 0" />
+        <mass value="0.03070001"/>
+        <inertia ixx="0.00012024" ixy="0.0"         ixz="0.0"
+                                   iyy="0.00012029" iyz="0.00000305"
+                                                    izz="0.00000216"/>
+        </inertial>
+      </xacro:unless>
+      <xacro:if value="${is_right}">
+        <!-- Right lower leg inertia -->
+        <inertial>
+        <origin xyz="0.0 0.00787644 -0.08928215" rpy="0 0 0" />
+        <mass value="0.03070001"/>
+        <inertia ixx="0.00012024" ixy="0.0"         ixz="0.0"
+                                   iyy="0.00012029" iyz="-0.00000305"
+                                                    izz="0.00000216"/>
+        </inertial>
+      </xacro:if>
       <!-- LOWER LEG LINK VISUAL -->
       <visual>
-        <origin rpy="0 0 0" xyz="0 0 0"/>
+        <origin xyz="0 0 0" rpy="0 0 0" />
         <geometry>
           <xacro:unless value="${is_right}">
@@ -147,5 +166,5 @@
       <!-- LOWER LEG LINK COLLISION -->
       <collision>
-        <origin rpy="0 0 0" xyz="0 0 0"/>
+        <origin xyz="0 0 0" rpy="0 0 0" />
         <geometry>
           <xacro:unless value="${is_right}">
@@ -179,15 +198,15 @@
     <link name="${prefix}_FOOT">
       <!-- FOOT INERTIAL -->
+      <!-- This link is symmetrical left or right -->
       <inertial>
-        <origin rpy="0 0 0" xyz="0 0 0"/>
-        <mass value="0.01"/>
-        <inertia ixy="0.0" ixz="0.0" iyz="0.0"
-          ixx="0.0"
-          iyy="0.0"
-          izz="0.0"/>
+        <origin xyz="0 0 0.00035767" rpy="0 0 0" />
+        <mass value="0.00693606"/>
+        <inertia ixx="0.00000057" ixy="0.0"         ixz="0.0"
+                                   iyy="0.00000084" iyz="0.0"
+                                                    izz="0.00000053"/>
      </inertial>
       <!-- FOOT VISUAL -->
       <visual>
-        <origin rpy="0 0 0" xyz="0 0 0"/>
+        <origin xyz="0 0 0" rpy="0 0 0" />
         <geometry>
           <mesh filename="package://robot_properties_quadruped/meshes/${mesh_ext}/with_foot/quadruped_foot.${mesh_ext}"/>
@@ -199,5 +218,5 @@
       <!-- FOOT COLLISION -->
       <collision>
-        <origin rpy="0 0 0" xyz="0 0 0"/>
+        <origin xyz="0 0 0" rpy="0 0 0" />
         <geometry>
             <mesh filename="package://robot_properties_quadruped/meshes/${mesh_ext}/with_foot/quadruped_foot.${mesh_ext}"/>

File: xacro/quadruped.urdf.xacro (robot description, xacro)
@@ -1,4 +1,4 @@
 <?xml version="1.0" ?>
-<robot name="quadruped"
+<robot name="solo"
   xmlns:controller="http://playerstage.sourceforge.net/gazebo/xmlschema/#controller"
   xmlns:interface="http://playerstage.sourceforge.net/gazebo/xmlschema/#interface"
@@ -9,23 +9,19 @@
   <xacro:property name="opacity" value="1.0" />
   <xacro:property name="mesh_ext" value="obj" />
-  <!-- Inertia computation -->
-  <xacro:property name="base_w" value=".2" />
-  <xacro:property name="base_l" value=".4" />
-  <xacro:property name="base_h" value=".05" />
-  <xacro:property name="base_m" value="2.0" />
+  <!-- This file is based on: https://atlas.is.localnet/confluence/display/AMDW/Quadruped+URDF+Files -->
   <link name="base_link">
     <!-- BASE LINK INERTIAL -->
     <inertial>
-        <origin rpy="0 0 0" xyz="0 0 0"/>
-        <mass value="${base_m}"/>
-        <inertia ixx="${1./12. * base_m * (base_h*base_h + base_w*base_w)}"
-                 iyy="${1./12. * base_m * (base_h*base_h + base_l*base_l)}"
-                 izz="${1./12. * base_m * (base_w*base_w + base_l*base_l)}"
-                 ixy="0" ixz="0" iyz="0"
+        <origin xyz="0 0 0" rpy="0 0 0" />
+        <mass value="1.43315091"/>
+        <!-- The base is extremely symmetrical. -->
+        <inertia ixx="0.00578574" ixy="0.0" ixz="0.0"
+                                  iyy="0.01938108" iyz="0.0"
+                                                   izz="0.02476124"
         />
     </inertial>
     <!-- BASE LINK VISUAL -->
     <visual>
-        <origin rpy="0 0 0" xyz="0 0 0"/>
+        <origin xyz="0 0 0" rpy="0 0 0" />
         <geometry>
           <mesh filename="package://robot_properties_quadruped/meshes/${mesh_ext}/with_foot/quadruped_body.${mesh_ext}"/>
@@ -37,5 +33,5 @@
     <!-- BASE LINK COLLISION -->
     <collision>
-        <origin rpy="0 0 0" xyz="0 0 0"/>
+        <origin xyz="0 0 0" rpy="0 0 0" />
         <geometry>
           <mesh filename="package://robot_properties_quadruped/meshes/${mesh_ext}/with_foot/quadruped_body.${mesh_ext}"/>

Commit message: rename everything to fit the solo name

File: xacro/leg.xacro (robot description, xacro)
@@ -69,8 +69,8 @@
         <geometry>
           <xacro:unless value="${is_right}">
-            <mesh filename="package://robot_properties_quadruped/meshes/${mesh_ext}/with_foot/quadruped_upper_leg_left_side.${mesh_ext}"/>
-          </xacro:unless>
-          <xacro:if value="${is_right}">
-            <mesh filename="package://robot_properties_quadruped/meshes/${mesh_ext}/with_foot/quadruped_upper_leg_right_side.${mesh_ext}"/>
+            <mesh filename="package://robot_properties_solo/meshes/${mesh_ext}/with_foot/solo_upper_leg_left_side.${mesh_ext}"/>
+          </xacro:unless>
+          <xacro:if value="${is_right}">
+            <mesh filename="package://robot_properties_solo/meshes/${mesh_ext}/with_foot/solo_upper_leg_right_side.${mesh_ext}"/>
           </xacro:if>
         </geometry>
@@ -84,8 +84,8 @@
         <geometry>
           <xacro:unless value="${is_right}">
-            <mesh filename="package://robot_properties_quadruped/meshes/${mesh_ext}/with_foot/quadruped_upper_leg_left_side.${mesh_ext}"/>
-          </xacro:unless>
-          <xacro:if value="${is_right}">
-            <mesh filename="package://robot_properties_quadruped/meshes/${mesh_ext}/with_foot/quadruped_upper_leg_right_side.${mesh_ext}"/>
+            <mesh filename="package://robot_properties_solo/meshes/${mesh_ext}/with_foot/solo_upper_leg_left_side.${mesh_ext}"/>
+          </xacro:unless>
+          <xacro:if value="${is_right}">
+            <mesh filename="package://robot_properties_solo/meshes/${mesh_ext}/with_foot/solo_upper_leg_right_side.${mesh_ext}"/>
           </xacro:if>
         </geometry>
@@ -154,8 +154,8 @@
         <geometry>
           <xacro:unless value="${is_right}">
-            <mesh filename="package://robot_properties_quadruped/meshes/${mesh_ext}/with_foot/quadruped_lower_leg_left_side.${mesh_ext}"/>
-          </xacro:unless>
-          <xacro:if value="${is_right}">
-            <mesh filename="package://robot_properties_quadruped/meshes/${mesh_ext}/with_foot/quadruped_lower_leg_right_side.${mesh_ext}"/>
+            <mesh filename="package://robot_properties_solo/meshes/${mesh_ext}/with_foot/solo_lower_leg_left_side.${mesh_ext}"/>
+          </xacro:unless>
+          <xacro:if value="${is_right}">
+            <mesh filename="package://robot_properties_solo/meshes/${mesh_ext}/with_foot/solo_lower_leg_right_side.${mesh_ext}"/>
           </xacro:if>
         </geometry>
@@ -169,8 +169,8 @@
         <geometry>
           <xacro:unless value="${is_right}">
-            <mesh filename="package://robot_properties_quadruped/meshes/${mesh_ext}/with_foot/quadruped_lower_leg_left_side.${mesh_ext}"/>
-          </xacro:unless>
-          <xacro:if value="${is_right}">
-            <mesh filename="package://robot_properties_quadruped/meshes/${mesh_ext}/with_foot/quadruped_lower_leg_right_side.${mesh_ext}"/>
+            <mesh filename="package://robot_properties_solo/meshes/${mesh_ext}/with_foot/solo_lower_leg_left_side.${mesh_ext}"/>
+          </xacro:unless>
+          <xacro:if value="${is_right}">
+            <mesh filename="package://robot_properties_solo/meshes/${mesh_ext}/with_foot/solo_lower_leg_right_side.${mesh_ext}"/>
           </xacro:if>
         </geometry>
@@ -210,5 +210,5 @@
         <origin xyz="0 0 0" rpy="0 0 0" />
         <geometry>
-          <mesh filename="package://robot_properties_quadruped/meshes/${mesh_ext}/with_foot/quadruped_foot.${mesh_ext}"/>
+          <mesh filename="package://robot_properties_solo/meshes/${mesh_ext}/with_foot/solo_foot.${mesh_ext}"/>
         </geometry>
         <material name="${color_name}">
@@ -220,5 +220,5 @@
         <origin xyz="0 0 0" rpy="0 0 0" />
         <geometry>
-            <mesh filename="package://robot_properties_quadruped/meshes/${mesh_ext}/with_foot/quadruped_foot.${mesh_ext}"/>
+            <mesh filename="package://robot_properties_solo/meshes/${mesh_ext}/with_foot/solo_foot.${mesh_ext}"/>
         </geometry>
         <material name="${color_name}">

File: xacro/plane_with_restitution.urdf.xacro (robot description, xacro)
@@ -14,5 +14,5 @@
       <origin rpy="0 0 0" xyz="0 0 0"/>
       <geometry>
-      <mesh filename="package://robot_properties_quadruped/meshes/plane.obj" scale="1 1 1"/>
+      <mesh filename="package://robot_properties_solo/meshes/plane.obj" scale="1 1 1"/>
       </geometry>
        <material name="white">

File: xacro/solo.urdf.xacro (robot description, xacro)
@@ -25,5 +25,5 @@
         <origin xyz="0 0 0" rpy="0 0 0" />
         <geometry>
-          <mesh filename="package://robot_properties_quadruped/meshes/${mesh_ext}/with_foot/quadruped_body.${mesh_ext}"/>
+          <mesh filename="package://robot_properties_solo/meshes/${mesh_ext}/with_foot/solo_body.${mesh_ext}"/>
         </geometry>
         <material name="${color_name}">
@@ -35,5 +35,5 @@
         <origin xyz="0 0 0" rpy="0 0 0" />
         <geometry>
-          <mesh filename="package://robot_properties_quadruped/meshes/${mesh_ext}/with_foot/quadruped_body.${mesh_ext}"/>
+          <mesh filename="package://robot_properties_solo/meshes/${mesh_ext}/with_foot/solo_body.${mesh_ext}"/>
         </geometry>
         <material name="${color_name}">

File: xacro/solo_old.urdf.xacro (robot description, xacro)
@@ -1,4 +1,4 @@
 <?xml version="1.0" ?>
-<robot name="quadruped"
+<robot name="solo"
   xmlns:controller="http://playerstage.sourceforge.net/gazebo/xmlschema/#controller"
   xmlns:interface="http://playerstage.sourceforge.net/gazebo/xmlschema/#interface"
@@ -27,5 +27,5 @@
         <geometry>
           <!-- <cylinder length="${upper_leg_length}" radius="${upper_leg_radius}"/> -->
-          <mesh filename="package://robot_properties_quadruped/meshes/cylinder.obj" scale="${upper_leg_radius} ${upper_leg_radius} ${upper_leg_length}"/>
+          <mesh filename="package://robot_properties_solo/meshes/cylinder.obj" scale="${upper_leg_radius} ${upper_leg_radius} ${upper_leg_length}"/>
         </geometry>
         <material name="grey">
@@ -65,5 +65,5 @@
         <geometry>
           <!-- <cylinder length="${upper_leg_length}" radius="${upper_leg_radius}"/> -->
-          <mesh filename="package://robot_properties_quadruped/meshes/cylinder.obj" scale="${upper_leg_radius} ${upper_leg_radius} ${upper_leg_length}"/>
+          <mesh filename="package://robot_properties_solo/meshes/cylinder.obj" scale="${upper_leg_radius} ${upper_leg_radius} ${upper_leg_length}"/>
         </geometry>
         <material name="grey">
@@ -100,5 +100,5 @@
         <geometry>
           <!-- <sphere radius="${upper_leg_radius}"/> -->
-          <mesh filename="package://robot_properties_quadruped/meshes/sphere.obj" scale="${upper_leg_radius} ${upper_leg_radius} ${upper_leg_radius}"/>
+          <mesh filename="package://robot_properties_solo/meshes/sphere.obj" scale="${upper_leg_radius} ${upper_leg_radius} ${upper_leg_radius}"/>
         </geometry>
         <material name="red">
@@ -134,5 +134,5 @@
         <origin rpy="0 0 0" xyz="0 0 0"/>
         <geometry>
-          <mesh filename="package://robot_properties_quadruped/meshes/cube.obj" scale="${base_l} ${base_w} ${base_h}"/>
+          <mesh filename="package://robot_properties_solo/meshes/cube.obj" scale="${base_l} ${base_w} ${base_h}"/>
         </geometry>
         <material name="white">

Commit message: Adding solo12: Extra DOF at the shoulders, 150 g extra at each shoulder. Including demo file to display robot.

File: xacro/leg.xacro (robot description, xacro)
@@ -7,39 +7,88 @@
   <xacro:property name="HFE_2_KFE_y" value="${37.45 * 0.001}" />
   <xacro:property name="HFE_2_KFE_z" value="${160.00 * 0.001}" />
-  <!-- To check this data to get the center of the foot properly -->
-  <xacro:property name="KFE_2_FOOT_y" value="${0.5 * 27.00 * 0.001}" />
+  <xacro:property name="KFE_2_FOOT_y" value="${8.0 * 0.001}" />
   <xacro:property name="KFE_2_FOOT_z" value="${160.00 * 0.001}" />
-  <xacro:property name="KFE_2_contact_y" value="${0 * 0.001}" />
-  <xacro:property name="KFE_2_contact_z" value="${(160.00 + 0.5*27) * 0.001}" />
-  <!-- This macro has for purpose to define a left leg -->
-  <xacro:macro name="leg" params="prefix is_front is_right mesh_ext
-                                  color_name color opacity">
-    <!-- Joint between the base and the ${prefix} upper leg -->
-    <joint name="${prefix}_HFE" type="revolute">
-      <parent link="base_link"/>
-      <child link="${prefix}_UPPER_LEG"/>
-      <limit effort="1000" lower="-10" upper="10" velocity="1000"/>
-      <!-- joints rotates around the y-axis -->
-      <axis xyz="0 1 0"/>
-      <!-- placement of the joint -->
-      <xacro:if value="${is_front}">
-        <xacro:unless value="${is_right}">
-          <origin xyz="${base_2_HFE_x} ${base_2_HFE_y} 0" rpy="0 0 0" />
-        </xacro:unless>
-        <xacro:if value="${is_right}">
-          <origin xyz="${base_2_HFE_x} ${-base_2_HFE_y} 0" rpy="0 0 0" />
-        </xacro:if>
-      </xacro:if>
-      <xacro:unless value="${is_front}">
-        <xacro:unless value="${is_right}">
-          <origin xyz="${-base_2_HFE_x} ${base_2_HFE_y} 0" rpy="0 0 0" />
-        </xacro:unless>
-        <xacro:if value="${is_right}">
-          <origin xyz="${-base_2_HFE_x} ${-base_2_HFE_y} 0" rpy="0 0 0" />
-        </xacro:if>
-      </xacro:unless>
-      <!-- pybullet simulation parameters -->
-      <dynamics damping="0.0" friction="0.0"/>
-    </joint>
+  <!-- Macro defining solo leg. -->
+  <xacro:macro name="leg" params="prefix is_front is_right has_side_motion
+                                  mesh_ext color_name color opacity">
+    <xacro:if value="${has_side_motion}">
+      <joint name="${prefix}_HAA" type="revolute">
+        <parent link="base_link"/>
+        <child link="${prefix}_SHOULDER"/>
+        <limit effort="1000" lower="-10" upper="10" velocity="1000"/>
+        <!-- joints rotates around the x-axis -->
+        <axis xyz="1 0 0"/>
+        <!-- placement of the joint -->
+        <xacro:if value="${is_front}">
+          <xacro:unless value="${is_right}">
+            <origin xyz="${base_2_HFE_x} ${base_2_HFE_y} 0" rpy="0 0 0" />
+          </xacro:unless>
+          <xacro:if value="${is_right}">
+            <origin xyz="${base_2_HFE_x} ${-base_2_HFE_y} 0" rpy="0 0 0" />
+          </xacro:if>
+        </xacro:if>
+        <xacro:unless value="${is_front}">
+          <xacro:unless value="${is_right}">
+            <origin xyz="${-base_2_HFE_x} ${base_2_HFE_y} 0" rpy="0 0 0" />
+          </xacro:unless>
+          <xacro:if value="${is_right}">
+            <origin xyz="${-base_2_HFE_x} ${-base_2_HFE_y} 0" rpy="0 0 0" />
+          </xacro:if>
+        </xacro:unless>
+        <!-- pybullet simulation parameters -->
+        <dynamics damping="0.0" friction="0.0"/>
+      </joint>
+      <link name="${prefix}_SHOULDER">
+        <!-- create a dummy shoulder link to join the two joints -->
+        <inertial>
+          <origin xyz="0. 0. 0." rpy="0 0 0" />
+          <!-- Adding extra weight for actuator module at shoulder. -->
+          <mass value="0.150"/>
+          <inertia ixx="0.00000001" ixy="0.0"        ixz="0.0"
+                                    iyy="0.00000001" iyz="0"
+                                                     izz="0.00000001"/>
+          </inertial>
+      </link>
+      <joint name="${prefix}_HFE" type="revolute">
+        <parent link="${prefix}_SHOULDER"/>
+        <child link="${prefix}_UPPER_LEG"/>
+        <limit effort="1000" lower="-10" upper="10" velocity="1000"/>
+        <!-- joints rotates around the y-axis -->
+        <axis xyz="0 1 0"/>
+        <!-- placement of the joint -->
+        <origin xyz="0 0 0" rpy="0 0 0" />
+        <!-- pybullet simulation parameters -->
+        <dynamics damping="0.0" friction="0.0"/>
+      </joint>
+    </xacro:if>
+    <xacro:unless value="${has_side_motion}">
+      <!-- Joint between the base and the ${prefix} upper leg -->
+      <joint name="${prefix}_HFE" type="revolute">
+        <parent link="base_link"/>
+        <child link="${prefix}_UPPER_LEG"/>
+        <limit effort="1000" lower="-10" upper="10" velocity="1000"/>
+        <!-- joints rotates around the y-axis -->
+        <axis xyz="0 1 0"/>
+        <!-- placement of the joint -->
+        <xacro:if value="${is_front}">
+          <xacro:unless value="${is_right}">
+            <origin xyz="${base_2_HFE_x} ${base_2_HFE_y} 0" rpy="0 0 0" />
+          </xacro:unless>
+          <xacro:if value="${is_right}">
+            <origin xyz="${base_2_HFE_x} ${-base_2_HFE_y} 0" rpy="0 0 0" />
+          </xacro:if>
+        </xacro:if>
+        <xacro:unless value="${is_front}">
+          <xacro:unless value="${is_right}">
+            <origin xyz="${-base_2_HFE_x} ${base_2_HFE_y} 0" rpy="0 0 0" />
+          </xacro:unless>
+          <xacro:if value="${is_right}">
+            <origin xyz="${-base_2_HFE_x} ${-base_2_HFE_y} 0" rpy="0 0 0" />
+          </xacro:if>
+        </xacro:unless>
+        <!-- pybullet simulation parameters -->
+        <dynamics damping="0.0" friction="0.0"/>
+      </joint>
+    </xacro:unless>
     <link name="${prefix}_UPPER_LEG">
       <!-- UPPER LEG LINK INERTIAL -->
@@ -190,5 +239,10 @@
       <child link="${prefix}_FOOT"/>
       <!-- Joint placement -->
-      <origin xyz="0 0 ${-HFE_2_KFE_z}" rpy="0 0 0" />
+      <xacro:unless value="${is_right}">
+        <origin xyz="0 ${KFE_2_FOOT_y} ${-KFE_2_FOOT_z}" rpy="0 0 0" />
+      </xacro:unless>
+      <xacro:if value="${is_right}">
+        <origin xyz="0 ${-KFE_2_FOOT_y} ${-KFE_2_FOOT_z}" rpy="0 0 0" />
+      </xacro:if>
       <!-- Limits (usefull?) -->
       <limit effort="1000" lower="-10" upper="10" velocity="1000"/>

File: xacro/solo12.urdf.xacro (robot description, xacro)
@@ -14,5 +14,5 @@
     <inertial>
         <origin xyz="0 0 0" rpy="0 0 0" />
-        <mass value="1.43315091"/>
+        <mass value="1.63315091"/>
         <!-- The base is extremely symmetrical. -->
         <inertia ixx="0.00578574" ixy="0.0" ixz="0.0"
@@ -54,5 +54,5 @@
       is_front="true"
       is_right="false"
-      has_side_motion="false"
+      has_side_motion="true"
       mesh_ext="${mesh_ext}"
       color_name="${color_name}"
@@ -64,5 +64,5 @@
       is_front="true"
       is_right="true"
-      has_side_motion="false"
+      has_side_motion="true"
       mesh_ext="${mesh_ext}"
       color_name="${color_name}"
@@ -74,5 +74,5 @@
       is_front="false"
       is_right="false"
-      has_side_motion="false"
+      has_side_motion="true"
       mesh_ext="${mesh_ext}"
       color_name="${color_name}"
@@ -84,5 +84,5 @@
       is_front="false"
       is_right="true"
-      has_side_motion="false"
+      has_side_motion="true"
       mesh_ext="${mesh_ext}"
       color_name="${color_name}"
