Commit message: Update solo12 to match closer latest real robot iteration

File: xacro/leg.xacro (robot description, xacro)
@@ -3,4 +3,7 @@
   <!-- See TODO: add the wiki link here -->
   <!-- These are absoulte distance value, the sign are decided below -->
+  <xacro:property name="base_2_HAA_x" value="${194.60 * 0.001}" />
+  <xacro:property name="base_2_HAA_y" value="${101.50 * 0.001}" />
+  <xacro:property name="HAA_2_HFE_y" value="${14.0 * 0.001}" />
   <xacro:property name="base_2_HFE_x" value="${190.00 * 0.001}" />
   <xacro:property name="base_2_HFE_y" value="${104.60 * 0.001}" />
@@ -22,16 +25,16 @@
         <xacro:if value="${is_front}">
           <xacro:unless value="${is_right}">
-            <origin xyz="${base_2_HFE_x} ${base_2_HFE_y} 0" rpy="0 0 0" />
-          </xacro:unless>
-          <xacro:if value="${is_right}">
-            <origin xyz="${base_2_HFE_x} ${-base_2_HFE_y} 0" rpy="0 0 0" />
+            <origin xyz="${base_2_HAA_x} ${base_2_HAA_y} 0" rpy="0 0 0" />
+          </xacro:unless>
+          <xacro:if value="${is_right}">
+            <origin xyz="${base_2_HAA_x} ${-base_2_HAA_y} 0" rpy="0 0 0" />
           </xacro:if>
         </xacro:if>
         <xacro:unless value="${is_front}">
           <xacro:unless value="${is_right}">
-            <origin xyz="${-base_2_HFE_x} ${base_2_HFE_y} 0" rpy="0 0 0" />
-          </xacro:unless>
-          <xacro:if value="${is_right}">
-            <origin xyz="${-base_2_HFE_x} ${-base_2_HFE_y} 0" rpy="0 0 0" />
+            <origin xyz="${-base_2_HAA_x} ${base_2_HAA_y} 0" rpy="0 0 0" />
+          </xacro:unless>
+          <xacro:if value="${is_right}">
+            <origin xyz="${-base_2_HAA_x} ${-base_2_HAA_y} 0" rpy="0 0 0" />
           </xacro:if>
         </xacro:unless>
@@ -40,13 +43,26 @@
       </joint>
       <link name="${prefix}_SHOULDER">
+        <!-- TODO: Update inertias and add visuals for link. -->
         <!-- create a dummy shoulder link to join the two joints -->
-        <inertial>
-          <origin xyz="0. 0. 0." rpy="0 0 0" />
-          <!-- Adding extra weight for actuator module at shoulder. -->
-          <mass value="0.150"/>
-          <inertia ixx="0.00000001" ixy="0.0"        ixz="0.0"
-                                    iyy="0.00000001" iyz="0"
-                                                     izz="0.00000001"/>
+        <xacro:unless value="${is_right}">
+          <!-- Left upper leg inertia -->
+          <inertial>
+          <origin xyz="-0.07870700 0.01 0." rpy="0 0 0" />
+          <mass value="0.14853845"/>
+          <inertia ixx="0.00003024" ixy="0.00004671" ixz="0.0"
+                                    iyy="0.00041193" iyz="0.0"
+                                                     izz="0.00041107"/>
           </inertial>
+        </xacro:unless>
+        <xacro:if value="${is_right}">
+          <!-- Right upper leg inertia -->
+          <inertial>
+          <origin xyz="-0.07870700 -0.01 0." rpy="0 0 0" />
+          <mass value="0.14853845"/>
+          <inertia ixx="0.00003024" ixy="-0.00004671" ixz="0.0"
+                                    iyy="0.00041193" iyz="0.0"
+                                                     izz="0.00041107"/>
+          </inertial>
+        </xacro:if>
       </link>
       <joint name="${prefix}_HFE" type="revolute">
@@ -57,5 +73,10 @@
         <axis xyz="0 1 0"/>
         <!-- placement of the joint -->
-        <origin xyz="0 0 0" rpy="0 0 0" />
+        <xacro:if value="${is_right}">
+          <origin xyz="0 ${-HAA_2_HFE_y} 0" rpy="0 0 0" />
+        </xacro:if>
+        <xacro:unless value="${is_right}">
+          <origin xyz="0 ${HAA_2_HFE_y} 0" rpy="0 0 0" />
+        </xacro:unless>
         <!-- pybullet simulation parameters -->
         <dynamics damping="0.0" friction="0.0"/>

Commit message: Fixing com for HAA on the back robot part

File: xacro/leg.xacro (robot description, xacro)
@@ -45,24 +45,39 @@
         <!-- TODO: Update inertias and add visuals for link. -->
         <!-- create a dummy shoulder link to join the two joints -->
-        <xacro:unless value="${is_right}">
-          <!-- Left upper leg inertia -->
-          <inertial>
-          <origin xyz="-0.07870700 0.01 0." rpy="0 0 0" />
+        <inertial>
           <mass value="0.14853845"/>
-          <inertia ixx="0.00003024" ixy="0.00004671" ixz="0.0"
-                                    iyy="0.00041193" iyz="0.0"
-                                                     izz="0.00041107"/>
-          </inertial>
-        </xacro:unless>
-        <xacro:if value="${is_right}">
-          <!-- Right upper leg inertia -->
-          <inertial>
-          <origin xyz="-0.07870700 -0.01 0." rpy="0 0 0" />
-          <mass value="0.14853845"/>
-          <inertia ixx="0.00003024" ixy="-0.00004671" ixz="0.0"
-                                    iyy="0.00041193" iyz="0.0"
-                                                     izz="0.00041107"/>
-          </inertial>
-        </xacro:if>
+          <xacro:if value="${is_front}">
+            <xacro:unless value="${is_right}">
+              <!-- Left upper leg inertia -->
+              <origin xyz="-0.07870700 0.01 0." rpy="0 0 0" />
+              <inertia ixx="0.00003024" ixy="0.00004671" ixz="0.0"
+                                        iyy="0.00041193" iyz="0.0"
+                                                        izz="0.00041107"/>
+            </xacro:unless>
+            <xacro:if value="${is_right}">
+              <!-- Right upper leg inertia -->
+              <origin xyz="-0.07870700 -0.01 0." rpy="0 0 0" />
+              <inertia ixx="0.00003024" ixy="-0.00004671" ixz="0.0"
+                                        iyy="0.00041193" iyz="0.0"
+                                                        izz="0.00041107"/>
+            </xacro:if>
+          </xacro:if>
+          <xacro:unless value="${is_front}">
+            <xacro:unless value="${is_right}">
+              <!-- Left upper leg inertia -->
+              <origin xyz="0.07870700 0.01 0." rpy="0 0 0" />
+              <inertia ixx="0.00003024" ixy="0.00004671" ixz="0.0"
+                                        iyy="0.00041193" iyz="0.0"
+                                                        izz="0.00041107"/>
+            </xacro:unless>
+            <xacro:if value="${is_right}">
+              <!-- Right upper leg inertia -->
+              <origin xyz="0.07870700 -0.01 0." rpy="0 0 0" />
+              <inertia ixx="0.00003024" ixy="-0.00004671" ixz="0.0"
+                                        iyy="0.00041193" iyz="0.0"
+                                                        izz="0.00041107"/>
+            </xacro:if>
+          </xacro:unless>
+        </inertial>
       </link>
       <joint name="${prefix}_HFE" type="revolute">

Commit message: Fix distances for base_2_HAA_y

File: xacro/leg.xacro (robot description, xacro)
@@ -4,5 +4,5 @@
   <!-- These are absoulte distance value, the sign are decided below -->
   <xacro:property name="base_2_HAA_x" value="${194.60 * 0.001}" />
-  <xacro:property name="base_2_HAA_y" value="${101.50 * 0.001}" />
+  <xacro:property name="base_2_HAA_y" value="${87.50 * 0.001}" />
   <xacro:property name="HAA_2_HFE_y" value="${14.0 * 0.001}" />
   <xacro:property name="base_2_HFE_x" value="${190.00 * 0.001}" />

Commit message: Add the meshes for solo12

File: xacro/leg.xacro (robot description, xacro)
@@ -43,6 +43,65 @@
       </joint>
       <link name="${prefix}_SHOULDER">
-        <!-- TODO: Update inertias and add visuals for link. -->
+        <!-- TODO: Update inertias. -->
         <!-- create a dummy shoulder link to join the two joints -->
+        <!-- HAA VISUAL -->
+        <visual>
+            <xacro:unless value="${is_right}">
+                <xacro:if value="${is_front}">
+                    <origin xyz="0.01950 0 0" rpy="0 0 0" />
+                    <geometry>
+                        <mesh filename="package://robot_properties_solo/meshes/${mesh_ext}/solo12/solo12_hip_fe_fl.${mesh_ext}"/>
+                    </geometry>
+                </xacro:if>
+                <xacro:unless value="${is_front}">
+                    <origin xyz="-0.01950 0 0" rpy="0 0 0" />
+                    <geometry>
+                        <mesh filename="package://robot_properties_solo/meshes/${mesh_ext}/solo12/solo12_hip_fe_hl.${mesh_ext}"/>
+                    </geometry>
+                </xacro:unless>
+            </xacro:unless>
+            <xacro:if value="${is_right}">
+                <xacro:if value="${is_front}">
+                    <origin xyz="0.01950 0 0" rpy="0 0 0" />
+                    <geometry>
+                        <mesh filename="package://robot_properties_solo/meshes/${mesh_ext}/solo12/solo12_hip_fe_fr.${mesh_ext}"/>
+                    </geometry>
+                </xacro:if>
+                <xacro:unless value="${is_front}">
+                    <origin xyz="-0.01950 0 0" rpy="0 0 0" />
+                    <geometry>
+                        <mesh filename="package://robot_properties_solo/meshes/${mesh_ext}/solo12/solo12_hip_fe_hr.${mesh_ext}"/>
+                    </geometry>
+                </xacro:unless>
+            </xacro:if>
+            <material name="${color_name}">
+                <color rgba="${color} ${opacity}"/>
+            </material>
+        </visual>
+        <!-- HAA LINK COLLISION -->
+        <collision>
+            <origin xyz="0 0 0" rpy="0 0 0" />
+            <geometry>
+                <xacro:unless value="${is_right}">
+                    <xacro:if value="${is_front}">
+                        <mesh filename="package://robot_properties_solo/meshes/${mesh_ext}/solo12/solo12_hip_fe_fl.${mesh_ext}"/>
+                    </xacro:if>
+                    <xacro:unless value="${is_front}">
+                        <mesh filename="package://robot_properties_solo/meshes/${mesh_ext}/solo12/solo12_hip_fe_hl.${mesh_ext}"/>
+                    </xacro:unless>
+                </xacro:unless>
+                <xacro:if value="${is_right}">
+                    <xacro:if value="${is_front}">
+                        <mesh filename="package://robot_properties_solo/meshes/${mesh_ext}/solo12/solo12_hip_fe_fr.${mesh_ext}"/>
+                    </xacro:if>
+                    <xacro:unless value="${is_front}">
+                        <mesh filename="package://robot_properties_solo/meshes/${mesh_ext}/solo12/solo12_hip_fe_hr.${mesh_ext}"/>
+                    </xacro:unless>
+                </xacro:if>
+            </geometry>
+            <material name="${color_name}">
+                <color rgba="${color} ${opacity}"/>
+            </material>
+        </collision>
         <inertial>
           <mass value="0.14853845"/>

File: xacro/solo12.urdf.xacro (robot description, xacro)
@@ -25,5 +25,5 @@
         <origin xyz="0 0 0" rpy="0 0 0" />
         <geometry>
-          <mesh filename="package://robot_properties_solo/meshes/${mesh_ext}/with_foot/solo_body.${mesh_ext}"/>
+          <mesh filename="package://robot_properties_solo/meshes/${mesh_ext}/solo12/solo_12_base.${mesh_ext}"/>
         </geometry>
         <material name="${color_name}">
@@ -35,5 +35,5 @@
         <origin xyz="0 0 0" rpy="0 0 0" />
         <geometry>
-          <mesh filename="package://robot_properties_solo/meshes/${mesh_ext}/with_foot/solo_body.${mesh_ext}"/>
+          <mesh filename="package://robot_properties_solo/meshes/${mesh_ext}/solo12/solo_12_base.${mesh_ext}"/>
         </geometry>
         <material name="${color_name}">

Commit message: fix the collision

File: xacro/leg.xacro (robot description, xacro)
@@ -81,23 +81,32 @@
         <!-- HAA LINK COLLISION -->
         <collision>
-            <origin xyz="0 0 0" rpy="0 0 0" />
-            <geometry>
                 <xacro:unless value="${is_right}">
-                    <xacro:if value="${is_front}">
+                <xacro:if value="${is_front}">
+                    <origin xyz="0.01950 0 0" rpy="0 0 0" />
+                    <geometry>
                         <mesh filename="package://robot_properties_solo/meshes/${mesh_ext}/solo12/solo12_hip_fe_fl.${mesh_ext}"/>
-                    </xacro:if>
-                    <xacro:unless value="${is_front}">
+                    </geometry>
+                </xacro:if>
+                <xacro:unless value="${is_front}">
+                    <origin xyz="-0.01950 0 0" rpy="0 0 0" />
+                    <geometry>
                         <mesh filename="package://robot_properties_solo/meshes/${mesh_ext}/solo12/solo12_hip_fe_hl.${mesh_ext}"/>
-                    </xacro:unless>
+                    </geometry>
                 </xacro:unless>
-                <xacro:if value="${is_right}">
-                    <xacro:if value="${is_front}">
+            </xacro:unless>
+            <xacro:if value="${is_right}">
+                <xacro:if value="${is_front}">
+                    <origin xyz="0.01950 0 0" rpy="0 0 0" />
+                    <geometry>
                         <mesh filename="package://robot_properties_solo/meshes/${mesh_ext}/solo12/solo12_hip_fe_fr.${mesh_ext}"/>
-                    </xacro:if>
-                    <xacro:unless value="${is_front}">
+                    </geometry>
+                </xacro:if>
+                <xacro:unless value="${is_front}">
+                    <origin xyz="-0.01950 0 0" rpy="0 0 0" />
+                    <geometry>
                         <mesh filename="package://robot_properties_solo/meshes/${mesh_ext}/solo12/solo12_hip_fe_hr.${mesh_ext}"/>
-                    </xacro:unless>
-                </xacro:if>
-            </geometry>
+                    </geometry>
+                </xacro:unless>
+            </xacro:if>
             <material name="${color_name}">
                 <color rgba="${color} ${opacity}"/>
@@ -108,5 +117,5 @@
           <xacro:if value="${is_front}">
             <xacro:unless value="${is_right}">
-              <!-- Left upper leg inertia -->
+              <!-- HAA body inertia -->
               <origin xyz="-0.07870700 0.01 0." rpy="0 0 0" />
               <inertia ixx="0.00003024" ixy="0.00004671" ixz="0.0"
@@ -115,5 +124,5 @@
             </xacro:unless>
             <xacro:if value="${is_right}">
-              <!-- Right upper leg inertia -->
+              <!-- HAA body inertia -->
               <origin xyz="-0.07870700 -0.01 0." rpy="0 0 0" />
               <inertia ixx="0.00003024" ixy="-0.00004671" ixz="0.0"
@@ -124,5 +133,5 @@
           <xacro:unless value="${is_front}">
             <xacro:unless value="${is_right}">
-              <!-- Left upper leg inertia -->
+              <!-- HAA body inertia -->
               <origin xyz="0.07870700 0.01 0." rpy="0 0 0" />
               <inertia ixx="0.00003024" ixy="0.00004671" ixz="0.0"
@@ -131,5 +140,5 @@
             </xacro:unless>
             <xacro:if value="${is_right}">
-              <!-- Right upper leg inertia -->
+              <!-- HAA body inertia -->
               <origin xyz="0.07870700 -0.01 0." rpy="0 0 0" />
               <inertia ixx="0.00003024" ixy="-0.00004671" ixz="0.0"
