Commit message: Make visual part of urdfs work with pybullet and pinocchio. Do so by creating a dummy link to the mesh folder inside the urdf folder for now.

File: urdf/plane_with_restitution.urdf (robot description, URDF)
Before this commit: robot plane, 1 links, 0 joints
Links:
- link planeLink: geometry collision box size=30 30 10; visual mesh filename=package://quadruped/meshes/plane.obj scale=1 1 1

Commit message: update teh config with some additionnal paramters

File: urdf/plane_with_restitution.urdf (robot description, URDF)
Before this commit: robot plane, 1 links, 0 joints
Links:
- link planeLink: geometry collision box size=30 30 10; visual mesh filename=package://robot_properties_quadruped/meshes/plane.obj scale=1 1 1
