Commit message: included package name explicitly in the urdf file; restructured folder/path. \n renamed yaml_path to dgm_yaml_path

File: src/robot_properties_solo/robot_properties_solo/xacro/leg.xacro (robot description, xacro)
@@ -51,5 +51,5 @@
                     <origin xyz="0.01950 0 0" rpy="0 0 0" />
                     <geometry>
-                        <mesh filename="package://meshes/${mesh_ext}/solo12/solo12_hip_fe_fl.${mesh_ext}"/>
+                        <mesh filename="package://robot_properties_solo/meshes/${mesh_ext}/solo12/solo12_hip_fe_fl.${mesh_ext}"/>
                     </geometry>
                 </xacro:if>
@@ -57,5 +57,5 @@
                     <origin xyz="-0.01950 0 0" rpy="0 0 0" />
                     <geometry>
-                        <mesh filename="package://meshes/${mesh_ext}/solo12/solo12_hip_fe_hl.${mesh_ext}"/>
+                        <mesh filename="package://robot_properties_solo/meshes/${mesh_ext}/solo12/solo12_hip_fe_hl.${mesh_ext}"/>
                     </geometry>
                 </xacro:unless>
@@ -65,5 +65,5 @@
                     <origin xyz="0.01950 0 0" rpy="0 0 0" />
                     <geometry>
-                        <mesh filename="package://meshes/${mesh_ext}/solo12/solo12_hip_fe_fr.${mesh_ext}"/>
+                        <mesh filename="package://robot_properties_solo/meshes/${mesh_ext}/solo12/solo12_hip_fe_fr.${mesh_ext}"/>
                     </geometry>
                 </xacro:if>
@@ -71,5 +71,5 @@
                     <origin xyz="-0.01950 0 0" rpy="0 0 0" />
                     <geometry>
-                        <mesh filename="package://meshes/${mesh_ext}/solo12/solo12_hip_fe_hr.${mesh_ext}"/>
+                        <mesh filename="package://robot_properties_solo/meshes/${mesh_ext}/solo12/solo12_hip_fe_hr.${mesh_ext}"/>
                     </geometry>
                 </xacro:unless>
@@ -85,5 +85,5 @@
                     <origin xyz="0.01950 0 0" rpy="0 0 0" />
                     <geometry>
-                        <mesh filename="package://meshes/${mesh_ext}/solo12/solo12_hip_fe_fl.${mesh_ext}"/>
+                        <mesh filename="package://robot_properties_solo/meshes/${mesh_ext}/solo12/solo12_hip_fe_fl.${mesh_ext}"/>
                     </geometry>
                 </xacro:if>
@@ -91,5 +91,5 @@
                     <origin xyz="-0.01950 0 0" rpy="0 0 0" />
                     <geometry>
-                        <mesh filename="package://meshes/${mesh_ext}/solo12/solo12_hip_fe_hl.${mesh_ext}"/>
+                        <mesh filename="package://robot_properties_solo/meshes/${mesh_ext}/solo12/solo12_hip_fe_hl.${mesh_ext}"/>
                     </geometry>
                 </xacro:unless>
@@ -99,5 +99,5 @@
                     <origin xyz="0.01950 0 0" rpy="0 0 0" />
                     <geometry>
-                        <mesh filename="package://meshes/${mesh_ext}/solo12/solo12_hip_fe_fr.${mesh_ext}"/>
+                        <mesh filename="package://robot_properties_solo/meshes/${mesh_ext}/solo12/solo12_hip_fe_fr.${mesh_ext}"/>
                     </geometry>
                 </xacro:if>
@@ -105,5 +105,5 @@
                     <origin xyz="-0.01950 0 0" rpy="0 0 0" />
                     <geometry>
-                        <mesh filename="package://meshes/${mesh_ext}/solo12/solo12_hip_fe_hr.${mesh_ext}"/>
+                        <mesh filename="package://robot_properties_solo/meshes/${mesh_ext}/solo12/solo12_hip_fe_hr.${mesh_ext}"/>
                     </geometry>
                 </xacro:unless>
@@ -222,8 +222,8 @@
         <geometry>
           <xacro:unless value="${is_right}">
-            <mesh filename="package://meshes/${mesh_ext}/with_foot/solo_upper_leg_left_side.${mesh_ext}"/>
-          </xacro:unless>
-          <xacro:if value="${is_right}">
-            <mesh filename="package://meshes/${mesh_ext}/with_foot/solo_upper_leg_right_side.${mesh_ext}"/>
+            <mesh filename="package://robot_properties_solo/meshes/${mesh_ext}/with_foot/solo_upper_leg_left_side.${mesh_ext}"/>
+          </xacro:unless>
+          <xacro:if value="${is_right}">
+            <mesh filename="package://robot_properties_solo/meshes/${mesh_ext}/with_foot/solo_upper_leg_right_side.${mesh_ext}"/>
           </xacro:if>
         </geometry>
@@ -237,8 +237,8 @@
         <geometry>
           <xacro:unless value="${is_right}">
-            <mesh filename="package://meshes/${mesh_ext}/with_foot/solo_upper_leg_left_side.${mesh_ext}"/>
-          </xacro:unless>
-          <xacro:if value="${is_right}">
-            <mesh filename="package://meshes/${mesh_ext}/with_foot/solo_upper_leg_right_side.${mesh_ext}"/>
+            <mesh filename="package://robot_properties_solo/meshes/${mesh_ext}/with_foot/solo_upper_leg_left_side.${mesh_ext}"/>
+          </xacro:unless>
+          <xacro:if value="${is_right}">
+            <mesh filename="package://robot_properties_solo/meshes/${mesh_ext}/with_foot/solo_upper_leg_right_side.${mesh_ext}"/>
           </xacro:if>
         </geometry>
@@ -307,8 +307,8 @@
         <geometry>
           <xacro:unless value="${is_right}">
-            <mesh filename="package://meshes/${mesh_ext}/with_foot/solo_lower_leg_left_side.${mesh_ext}"/>
-          </xacro:unless>
-          <xacro:if value="${is_right}">
-            <mesh filename="package://meshes/${mesh_ext}/with_foot/solo_lower_leg_right_side.${mesh_ext}"/>
+            <mesh filename="package://robot_properties_solo/meshes/${mesh_ext}/with_foot/solo_lower_leg_left_side.${mesh_ext}"/>
+          </xacro:unless>
+          <xacro:if value="${is_right}">
+            <mesh filename="package://robot_properties_solo/meshes/${mesh_ext}/with_foot/solo_lower_leg_right_side.${mesh_ext}"/>
           </xacro:if>
         </geometry>
@@ -322,8 +322,8 @@
         <geometry>
           <xacro:unless value="${is_right}">
-            <mesh filename="package://meshes/${mesh_ext}/with_foot/solo_lower_leg_left_side.${mesh_ext}"/>
-          </xacro:unless>
-          <xacro:if value="${is_right}">
-            <mesh filename="package://meshes/${mesh_ext}/with_foot/solo_lower_leg_right_side.${mesh_ext}"/>
+            <mesh filename="package://robot_properties_solo/meshes/${mesh_ext}/with_foot/solo_lower_leg_left_side.${mesh_ext}"/>
+          </xacro:unless>
+          <xacro:if value="${is_right}">
+            <mesh filename="package://robot_properties_solo/meshes/${mesh_ext}/with_foot/solo_lower_leg_right_side.${mesh_ext}"/>
           </xacro:if>
         </geometry>
@@ -368,5 +368,5 @@
         <origin xyz="0 0 0" rpy="0 0 0" />
         <geometry>
-          <mesh filename="package://meshes/${mesh_ext}/with_foot/solo_foot.${mesh_ext}"/>
+          <mesh filename="package://robot_properties_solo/meshes/${mesh_ext}/with_foot/solo_foot.${mesh_ext}"/>
         </geometry>
         <material name="${color_name}">
@@ -378,5 +378,5 @@
         <origin xyz="0 0 0" rpy="0 0 0" />
         <geometry>
-            <mesh filename="package://meshes/${mesh_ext}/with_foot/solo_foot.${mesh_ext}"/>
+            <mesh filename="package://robot_properties_solo/meshes/${mesh_ext}/with_foot/solo_foot.${mesh_ext}"/>
         </geometry>
         <material name="${color_name}">

File: src/robot_properties_solo/robot_properties_solo/xacro/plane_with_restitution.urdf.xacro (robot description, xacro)
@@ -14,5 +14,5 @@
       <origin rpy="0 0 0" xyz="0 0 0"/>
       <geometry>
-      <mesh filename="package://meshes/plane.obj" scale="1 1 1"/>
+      <mesh filename="package://robot_properties_solo/meshes/plane.obj" scale="1 1 1"/>
       </geometry>
        <material name="white">

File: src/robot_properties_solo/robot_properties_solo/xacro/solo12.urdf.xacro (robot description, xacro)
@@ -14,5 +14,5 @@
     <inertial>
         <origin xyz="0 0 0" rpy="0 0 0" />
-        <mass value="1.43315091"/>
+        <mass value="1.16115091"/>
         <!-- The base is extremely symmetrical. -->
         <inertia ixx="0.00578574" ixy="0.0" ixz="0.0"
@@ -25,5 +25,5 @@
         <origin xyz="0 0 0" rpy="0 0 0" />
         <geometry>
-          <mesh filename="package://meshes/${mesh_ext}/with_foot/solo_body.${mesh_ext}"/>
+          <mesh filename="package://robot_properties_solo/meshes/${mesh_ext}/solo12/solo_12_base.${mesh_ext}"/>
         </geometry>
         <material name="${color_name}">
@@ -35,5 +35,5 @@
         <origin xyz="0 0 0" rpy="0 0 0" />
         <geometry>
-          <mesh filename="package://meshes/${mesh_ext}/with_foot/solo_body.${mesh_ext}"/>
+          <mesh filename="package://robot_properties_solo/meshes/${mesh_ext}/solo12/solo_12_base.${mesh_ext}"/>
         </geometry>
         <material name="${color_name}">
@@ -54,5 +54,5 @@
       is_front="true"
       is_right="false"
-      has_side_motion="false"
+      has_side_motion="true"
       mesh_ext="${mesh_ext}"
       color_name="${color_name}"
@@ -64,5 +64,5 @@
       is_front="true"
       is_right="true"
-      has_side_motion="false"
+      has_side_motion="true"
       mesh_ext="${mesh_ext}"
       color_name="${color_name}"
@@ -74,5 +74,5 @@
       is_front="false"
       is_right="false"
-      has_side_motion="false"
+      has_side_motion="true"
       mesh_ext="${mesh_ext}"
       color_name="${color_name}"
@@ -84,5 +84,5 @@
       is_front="false"
       is_right="true"
-      has_side_motion="false"
+      has_side_motion="true"
       mesh_ext="${mesh_ext}"
       color_name="${color_name}"

File: src/robot_properties_solo/robot_properties_solo/xacro/solo8.urdf.xacro (robot description, xacro)
@@ -14,5 +14,5 @@
     <inertial>
         <origin xyz="0 0 0" rpy="0 0 0" />
-        <mass value="1.16115091"/>
+        <mass value="1.43315091"/>
         <!-- The base is extremely symmetrical. -->
         <inertia ixx="0.00578574" ixy="0.0" ixz="0.0"
@@ -25,5 +25,5 @@
         <origin xyz="0 0 0" rpy="0 0 0" />
         <geometry>
-          <mesh filename="package://meshes/${mesh_ext}/solo12/solo_12_base.${mesh_ext}"/>
+          <mesh filename="package://robot_properties_solo/meshes/${mesh_ext}/with_foot/solo_body.${mesh_ext}"/>
         </geometry>
         <material name="${color_name}">
@@ -35,5 +35,5 @@
         <origin xyz="0 0 0" rpy="0 0 0" />
         <geometry>
-          <mesh filename="package://meshes/${mesh_ext}/solo12/solo_12_base.${mesh_ext}"/>
+          <mesh filename="package://robot_properties_solo/meshes/${mesh_ext}/with_foot/solo_body.${mesh_ext}"/>
         </geometry>
         <material name="${color_name}">
@@ -54,5 +54,5 @@
       is_front="true"
       is_right="false"
-      has_side_motion="true"
+      has_side_motion="false"
       mesh_ext="${mesh_ext}"
       color_name="${color_name}"
@@ -64,5 +64,5 @@
       is_front="true"
       is_right="true"
-      has_side_motion="true"
+      has_side_motion="false"
       mesh_ext="${mesh_ext}"
       color_name="${color_name}"
@@ -74,5 +74,5 @@
       is_front="false"
       is_right="false"
-      has_side_motion="true"
+      has_side_motion="false"
       mesh_ext="${mesh_ext}"
       color_name="${color_name}"
@@ -84,5 +84,5 @@
       is_front="false"
       is_right="true"
-      has_side_motion="true"
+      has_side_motion="false"
       mesh_ext="${mesh_ext}"
       color_name="${color_name}"
