Commit message: build xacro files at installation time; rename resources folder to 'resources'

File: src/robot_properties_solo/resources/xacro/leg.xacro (robot description, xacro)
@@ -51,5 +51,5 @@
                     <origin xyz="0.01950 0 0" rpy="0 0 0" />
                     <geometry>
-                        <mesh filename="package://robot_properties_solo/meshes/${mesh_ext}/solo12/solo12_hip_fe_fl.${mesh_ext}"/>
+                        <mesh filename="package://robot_properties_solo/resources/meshes/${mesh_ext}/solo12/solo12_hip_fe_fl.${mesh_ext}"/>
                     </geometry>
                 </xacro:if>
@@ -57,5 +57,5 @@
                     <origin xyz="-0.01950 0 0" rpy="0 0 0" />
                     <geometry>
-                        <mesh filename="package://robot_properties_solo/meshes/${mesh_ext}/solo12/solo12_hip_fe_hl.${mesh_ext}"/>
+                        <mesh filename="package://robot_properties_solo/resources/meshes/${mesh_ext}/solo12/solo12_hip_fe_hl.${mesh_ext}"/>
                     </geometry>
                 </xacro:unless>
@@ -65,5 +65,5 @@
                     <origin xyz="0.01950 0 0" rpy="0 0 0" />
                     <geometry>
-                        <mesh filename="package://robot_properties_solo/meshes/${mesh_ext}/solo12/solo12_hip_fe_fr.${mesh_ext}"/>
+                        <mesh filename="package://robot_properties_solo/resources/meshes/${mesh_ext}/solo12/solo12_hip_fe_fr.${mesh_ext}"/>
                     </geometry>
                 </xacro:if>
@@ -71,5 +71,5 @@
                     <origin xyz="-0.01950 0 0" rpy="0 0 0" />
                     <geometry>
-                        <mesh filename="package://robot_properties_solo/meshes/${mesh_ext}/solo12/solo12_hip_fe_hr.${mesh_ext}"/>
+                        <mesh filename="package://robot_properties_solo/resources/meshes/${mesh_ext}/solo12/solo12_hip_fe_hr.${mesh_ext}"/>
                     </geometry>
                 </xacro:unless>
@@ -85,5 +85,5 @@
                     <origin xyz="0.01950 0 0" rpy="0 0 0" />
                     <geometry>
-                        <mesh filename="package://robot_properties_solo/meshes/${mesh_ext}/solo12/solo12_hip_fe_fl.${mesh_ext}"/>
+                        <mesh filename="package://robot_properties_solo/resources/meshes/${mesh_ext}/solo12/solo12_hip_fe_fl.${mesh_ext}"/>
                     </geometry>
                 </xacro:if>
@@ -91,5 +91,5 @@
                     <origin xyz="-0.01950 0 0" rpy="0 0 0" />
                     <geometry>
-                        <mesh filename="package://robot_properties_solo/meshes/${mesh_ext}/solo12/solo12_hip_fe_hl.${mesh_ext}"/>
+                        <mesh filename="package://robot_properties_solo/resources/meshes/${mesh_ext}/solo12/solo12_hip_fe_hl.${mesh_ext}"/>
                     </geometry>
                 </xacro:unless>
@@ -99,5 +99,5 @@
                     <origin xyz="0.01950 0 0" rpy="0 0 0" />
                     <geometry>
-                        <mesh filename="package://robot_properties_solo/meshes/${mesh_ext}/solo12/solo12_hip_fe_fr.${mesh_ext}"/>
+                        <mesh filename="package://robot_properties_solo/resources/meshes/${mesh_ext}/solo12/solo12_hip_fe_fr.${mesh_ext}"/>
                     </geometry>
                 </xacro:if>
@@ -105,5 +105,5 @@
                     <origin xyz="-0.01950 0 0" rpy="0 0 0" />
                     <geometry>
-                        <mesh filename="package://robot_properties_solo/meshes/${mesh_ext}/solo12/solo12_hip_fe_hr.${mesh_ext}"/>
+                        <mesh filename="package://robot_properties_solo/resources/meshes/${mesh_ext}/solo12/solo12_hip_fe_hr.${mesh_ext}"/>
                     </geometry>
                 </xacro:unless>
@@ -222,8 +222,8 @@
         <geometry>
           <xacro:unless value="${is_right}">
-            <mesh filename="package://robot_properties_solo/meshes/${mesh_ext}/with_foot/solo_upper_leg_left_side.${mesh_ext}"/>
-          </xacro:unless>
-          <xacro:if value="${is_right}">
-            <mesh filename="package://robot_properties_solo/meshes/${mesh_ext}/with_foot/solo_upper_leg_right_side.${mesh_ext}"/>
+            <mesh filename="package://robot_properties_solo/resources/meshes/${mesh_ext}/with_foot/solo_upper_leg_left_side.${mesh_ext}"/>
+          </xacro:unless>
+          <xacro:if value="${is_right}">
+            <mesh filename="package://robot_properties_solo/resources/meshes/${mesh_ext}/with_foot/solo_upper_leg_right_side.${mesh_ext}"/>
           </xacro:if>
         </geometry>
@@ -237,8 +237,8 @@
         <geometry>
           <xacro:unless value="${is_right}">
-            <mesh filename="package://robot_properties_solo/meshes/${mesh_ext}/with_foot/solo_upper_leg_left_side.${mesh_ext}"/>
-          </xacro:unless>
-          <xacro:if value="${is_right}">
-            <mesh filename="package://robot_properties_solo/meshes/${mesh_ext}/with_foot/solo_upper_leg_right_side.${mesh_ext}"/>
+            <mesh filename="package://robot_properties_solo/resources/meshes/${mesh_ext}/with_foot/solo_upper_leg_left_side.${mesh_ext}"/>
+          </xacro:unless>
+          <xacro:if value="${is_right}">
+            <mesh filename="package://robot_properties_solo/resources/meshes/${mesh_ext}/with_foot/solo_upper_leg_right_side.${mesh_ext}"/>
           </xacro:if>
         </geometry>
@@ -307,8 +307,8 @@
         <geometry>
           <xacro:unless value="${is_right}">
-            <mesh filename="package://robot_properties_solo/meshes/${mesh_ext}/with_foot/solo_lower_leg_left_side.${mesh_ext}"/>
-          </xacro:unless>
-          <xacro:if value="${is_right}">
-            <mesh filename="package://robot_properties_solo/meshes/${mesh_ext}/with_foot/solo_lower_leg_right_side.${mesh_ext}"/>
+            <mesh filename="package://robot_properties_solo/resources/meshes/${mesh_ext}/with_foot/solo_lower_leg_left_side.${mesh_ext}"/>
+          </xacro:unless>
+          <xacro:if value="${is_right}">
+            <mesh filename="package://robot_properties_solo/resources/meshes/${mesh_ext}/with_foot/solo_lower_leg_right_side.${mesh_ext}"/>
           </xacro:if>
         </geometry>
@@ -322,8 +322,8 @@
         <geometry>
           <xacro:unless value="${is_right}">
-            <mesh filename="package://robot_properties_solo/meshes/${mesh_ext}/with_foot/solo_lower_leg_left_side.${mesh_ext}"/>
-          </xacro:unless>
-          <xacro:if value="${is_right}">
-            <mesh filename="package://robot_properties_solo/meshes/${mesh_ext}/with_foot/solo_lower_leg_right_side.${mesh_ext}"/>
+            <mesh filename="package://robot_properties_solo/resources/meshes/${mesh_ext}/with_foot/solo_lower_leg_left_side.${mesh_ext}"/>
+          </xacro:unless>
+          <xacro:if value="${is_right}">
+            <mesh filename="package://robot_properties_solo/resources/meshes/${mesh_ext}/with_foot/solo_lower_leg_right_side.${mesh_ext}"/>
           </xacro:if>
         </geometry>
@@ -368,5 +368,5 @@
         <origin xyz="0 0 0" rpy="0 0 0" />
         <geometry>
-          <mesh filename="package://robot_properties_solo/meshes/${mesh_ext}/with_foot/solo_foot.${mesh_ext}"/>
+          <mesh filename="package://robot_properties_solo/resources/meshes/${mesh_ext}/with_foot/solo_foot.${mesh_ext}"/>
         </geometry>
         <material name="${color_name}">
@@ -378,5 +378,5 @@
         <origin xyz="0 0 0" rpy="0 0 0" />
         <geometry>
-            <mesh filename="package://robot_properties_solo/meshes/${mesh_ext}/with_foot/solo_foot.${mesh_ext}"/>
+            <mesh filename="package://robot_properties_solo/resources/meshes/${mesh_ext}/with_foot/solo_foot.${mesh_ext}"/>
         </geometry>
         <material name="${color_name}">

File: src/robot_properties_solo/resources/xacro/plane_with_restitution.urdf.xacro (robot description, xacro)
@@ -14,5 +14,5 @@
       <origin rpy="0 0 0" xyz="0 0 0"/>
       <geometry>
-      <mesh filename="package://robot_properties_solo/meshes/plane.obj" scale="1 1 1"/>
+      <mesh filename="package://robot_properties_solo/resources/meshes/plane.obj" scale="1 1 1"/>
       </geometry>
        <material name="white">

File: src/robot_properties_solo/resources/xacro/solo12.urdf.xacro (robot description, xacro)
@@ -14,5 +14,5 @@
     <inertial>
         <origin xyz="0 0 0" rpy="0 0 0" />
-        <mass value="1.43315091"/>
+        <mass value="1.16115091"/>
         <!-- The base is extremely symmetrical. -->
         <inertia ixx="0.00578574" ixy="0.0" ixz="0.0"
@@ -25,5 +25,5 @@
         <origin xyz="0 0 0" rpy="0 0 0" />
         <geometry>
-          <mesh filename="package://robot_properties_solo/meshes/${mesh_ext}/with_foot/solo_body.${mesh_ext}"/>
+          <mesh filename="package://robot_properties_solo/resources/meshes/${mesh_ext}/solo12/solo_12_base.${mesh_ext}"/>
         </geometry>
         <material name="${color_name}">
@@ -35,5 +35,5 @@
         <origin xyz="0 0 0" rpy="0 0 0" />
         <geometry>
-          <mesh filename="package://robot_properties_solo/meshes/${mesh_ext}/with_foot/solo_body.${mesh_ext}"/>
+          <mesh filename="package://robot_properties_solo/resources/meshes/${mesh_ext}/solo12/solo_12_base.${mesh_ext}"/>
         </geometry>
         <material name="${color_name}">
@@ -54,5 +54,5 @@
       is_front="true"
       is_right="false"
-      has_side_motion="false"
+      has_side_motion="true"
       mesh_ext="${mesh_ext}"
       color_name="${color_name}"
@@ -64,5 +64,5 @@
       is_front="true"
       is_right="true"
-      has_side_motion="false"
+      has_side_motion="true"
       mesh_ext="${mesh_ext}"
       color_name="${color_name}"
@@ -74,5 +74,5 @@
       is_front="false"
       is_right="false"
-      has_side_motion="false"
+      has_side_motion="true"
       mesh_ext="${mesh_ext}"
       color_name="${color_name}"
@@ -84,5 +84,5 @@
       is_front="false"
       is_right="true"
-      has_side_motion="false"
+      has_side_motion="true"
       mesh_ext="${mesh_ext}"
       color_name="${color_name}"

File: src/robot_properties_solo/resources/xacro/solo8.urdf.xacro (robot description, xacro)
@@ -14,5 +14,5 @@
     <inertial>
         <origin xyz="0 0 0" rpy="0 0 0" />
-        <mass value="1.16115091"/>
+        <mass value="1.43315091"/>
         <!-- The base is extremely symmetrical. -->
         <inertia ixx="0.00578574" ixy="0.0" ixz="0.0"
@@ -25,5 +25,5 @@
         <origin xyz="0 0 0" rpy="0 0 0" />
         <geometry>
-          <mesh filename="package://robot_properties_solo/meshes/${mesh_ext}/solo12/solo_12_base.${mesh_ext}"/>
+          <mesh filename="package://robot_properties_solo/resources/meshes/${mesh_ext}/with_foot/solo_body.${mesh_ext}"/>
         </geometry>
         <material name="${color_name}">
@@ -35,5 +35,5 @@
         <origin xyz="0 0 0" rpy="0 0 0" />
         <geometry>
-          <mesh filename="package://robot_properties_solo/meshes/${mesh_ext}/solo12/solo_12_base.${mesh_ext}"/>
+          <mesh filename="package://robot_properties_solo/resources/meshes/${mesh_ext}/with_foot/solo_body.${mesh_ext}"/>
         </geometry>
         <material name="${color_name}">
@@ -54,5 +54,5 @@
       is_front="true"
       is_right="false"
-      has_side_motion="true"
+      has_side_motion="false"
       mesh_ext="${mesh_ext}"
       color_name="${color_name}"
@@ -64,5 +64,5 @@
       is_front="true"
       is_right="true"
-      has_side_motion="true"
+      has_side_motion="false"
       mesh_ext="${mesh_ext}"
       color_name="${color_name}"
@@ -74,5 +74,5 @@
       is_front="false"
       is_right="false"
-      has_side_motion="true"
+      has_side_motion="false"
       mesh_ext="${mesh_ext}"
       color_name="${color_name}"
@@ -84,5 +84,5 @@
       is_front="false"
       is_right="true"
-      has_side_motion="true"
+      has_side_motion="false"
       mesh_ext="${mesh_ext}"
       color_name="${color_name}"

Commit message: update the leg and body xacro files

File: src/robot_properties_solo/resources/xacro/leg.xacro (robot description, xacro)
@@ -3,12 +3,13 @@
   <!-- See TODO: add the wiki link here -->
   <!-- These are absoulte distance value, the sign are decided below -->
-  <xacro:property name="base_2_HAA_x" value="${194.60 * 0.001}" />
+  <xacro:property name="base_2_HAA_x" value="${214.10 * 0.001}" />
   <xacro:property name="base_2_HAA_y" value="${87.50 * 0.001}" />
   <xacro:property name="HAA_2_HFE_y" value="${14.0 * 0.001}" />
-  <xacro:property name="base_2_HFE_x" value="${190.00 * 0.001}" />
-  <xacro:property name="base_2_HFE_y" value="${104.60 * 0.001}" />
+  <xacro:property name="HAA_2_HFE_x" value="${19.5 * 0.001}" />
+  <xacro:property name="base_2_HFE_x" value="${194.60 * 0.001}" />
+  <xacro:property name="base_2_HFE_y" value="${101.50 * 0.001}" />
   <xacro:property name="HFE_2_KFE_y" value="${37.45 * 0.001}" />
   <xacro:property name="HFE_2_KFE_z" value="${160.00 * 0.001}" />
-  <xacro:property name="KFE_2_FOOT_y" value="${8.0 * 0.001}" />
+  <xacro:property name="KFE_2_FOOT_y" value="${9.0 * 0.001}" />
   <xacro:property name="KFE_2_FOOT_z" value="${160.00 * 0.001}" />
   <!-- Macro defining solo leg. -->
@@ -114,19 +115,19 @@
         </collision>
         <inertial>
-          <mass value="0.14853845"/>
+          <mass value="0.14196048"/>
           <xacro:if value="${is_front}">
             <xacro:unless value="${is_right}">
               <!-- HAA body inertia -->
-              <origin xyz="-0.07870700 0.01 0." rpy="0 0 0" />
-              <inertia ixx="0.00003024" ixy="0.00004671" ixz="0.0"
-                                        iyy="0.00041193" iyz="0.0"
-                                                        izz="0.00041107"/>
+              <origin xyz="-0.09407251 -0.00438935 0.00001384" rpy="0 0 0" />
+              <inertia ixx="0.00002802" ixy="0.00003687" ixz="-0.00000009"
+                                        iyy="0.00038264" iyz="0.00000000"
+                                                         izz="0.00038050"/>
             </xacro:unless>
             <xacro:if value="${is_right}">
               <!-- HAA body inertia -->
-              <origin xyz="-0.07870700 -0.01 0." rpy="0 0 0" />
-              <inertia ixx="0.00003024" ixy="-0.00004671" ixz="0.0"
-                                        iyy="0.00041193" iyz="0.0"
-                                                        izz="0.00041107"/>
+              <origin xyz="-0.09407251 0.00438935 -0.00001384" rpy="0 0 0" />
+              <inertia ixx="0.00002802" ixy="-0.00003687" ixz="0.00000009"
+                                        iyy="0.00038264"  iyz="0.00000000"
+                                                          izz="0.00038050"/>
             </xacro:if>
           </xacro:if>
@@ -134,15 +135,15 @@
             <xacro:unless value="${is_right}">
               <!-- HAA body inertia -->
-              <origin xyz="0.07870700 0.01 0." rpy="0 0 0" />
-              <inertia ixx="0.00003024" ixy="0.00004671" ixz="0.0"
-                                        iyy="0.00041193" iyz="0.0"
-                                                        izz="0.00041107"/>
+              <origin xyz="0.09407251 -0.00438935 -0.00001384" rpy="0 0 0" />
+              <inertia ixx="0.00002802" ixy="-0.00003687" ixz="-0.00000009"
+                                        iyy="0.00038264"  iyz="0.00000000"
+                                                          izz="0.00038050"/>
             </xacro:unless>
             <xacro:if value="${is_right}">
               <!-- HAA body inertia -->
-              <origin xyz="0.07870700 -0.01 0." rpy="0 0 0" />
-              <inertia ixx="0.00003024" ixy="-0.00004671" ixz="0.0"
-                                        iyy="0.00041193" iyz="0.0"
-                                                        izz="0.00041107"/>
+              <origin xyz="0.09407251 0.00438935 0.00001384" rpy="0 0 0" />
+              <inertia ixx="0.00002802" ixy="0.00003687" ixz="0.00000009"
+                                        iyy="0.00038264" iyz="0.00000000"
+                                                         izz="0.00038050"/>
             </xacro:if>
           </xacro:unless>
@@ -156,9 +157,19 @@
         <axis xyz="0 1 0"/>
         <!-- placement of the joint -->
-        <xacro:if value="${is_right}">
-          <origin xyz="0 ${-HAA_2_HFE_y} 0" rpy="0 0 0" />
+        <xacro:if value="${is_front}">
+          <xacro:unless value="${is_right}">
+            <origin xyz="${-HAA_2_HFE_x} ${HAA_2_HFE_y} 0" rpy="0 0 0" />
+          </xacro:unless>
+          <xacro:if value="${is_right}">
+            <origin xyz="${-HAA_2_HFE_x} ${-HAA_2_HFE_y} 0" rpy="0 0 0" />
+          </xacro:if>
         </xacro:if>
-        <xacro:unless value="${is_right}">
-          <origin xyz="0 ${HAA_2_HFE_y} 0" rpy="0 0 0" />
+        <xacro:unless value="${is_front}">
+          <xacro:unless value="${is_right}">
+            <origin xyz="${HAA_2_HFE_x} ${HAA_2_HFE_y} 0" rpy="0 0 0" />
+          </xacro:unless>
+          <xacro:if value="${is_right}">
+            <origin xyz="${HAA_2_HFE_x} ${-HAA_2_HFE_y} 0" rpy="0 0 0" />
+          </xacro:if>
         </xacro:unless>
         <!-- pybullet simulation parameters -->
@@ -200,9 +211,9 @@
         <!-- Left upper leg inertia -->
         <inertial>
-        <origin xyz="0.00001377 0.01935853 -0.07870700" rpy="0 0 0" />
-        <mass value="0.14853845"/>
-        <inertia ixx="0.00041107" ixy="0.0"         ixz="0.0"
-                                   iyy="0.00041193" iyz="0.00004671"
-                                                    izz="0.00003024"/>
+        <mass value="0.14737324"/>
+        <origin xyz="0.00001530 0.01767640 -0.07838230" rpy="0 0 0" />
+        <inertia ixx="0.00041540"  ixy="0.00000000" ixz="0.00000010"
+                                   iyy="0.00041637" iyz="-0.00004589"
+                                                    izz="0.00002982"/>
         </inertial>
       </xacro:unless>
@@ -210,9 +221,9 @@
         <!-- Right upper leg inertia -->
         <inertial>
-        <origin xyz="-0.00001377 -0.01935853 -0.07870700" rpy="0 0 0" />
-        <mass value="0.14853845"/>
-        <inertia ixx="0.00041107" ixy="0.0"         ixz="0.0"
-                                   iyy="0.00041193" iyz="-0.00004671"
-                                                    izz="0.00003024"/>
+        <mass value="0.14737324"/>
+        <origin xyz="-0.00001530 -0.01767640 -0.07838230" rpy="0 0 0" />
+        <inertia ixx="0.00041540"  ixy="0.00000000" ixz="-0.00000010"
+                                   iyy="0.00041637" iyz="0.00004589"
+                                                    izz="0.00002982"/>
         </inertial>
       </xacro:if>
@@ -285,9 +296,9 @@
         <!-- Left lower leg inertia -->
         <inertial>
-        <origin xyz="0.0 0.00787644 -0.08928215" rpy="0 0 0" />
-        <mass value="0.03070001"/>
-        <inertia ixx="0.00012024" ixy="0.0"         ixz="0.0"
-                                   iyy="0.00012029" iyz="0.00000305"
-                                                    izz="0.00000216"/>
+        <mass value="0.02318294"/>
+        <origin xyz="0.00000000 0.00776716 -0.07003876" rpy="0 0 0" />
+        <inertia ixx="0.00008508" ixy="0.00000000"  ixz="0.00000000"
+                                  iyy="0.00008580"  iyz="-0.00000200"
+                                                    izz="0.00000139"/>
         </inertial>
       </xacro:unless>
@@ -295,9 +306,9 @@
         <!-- Right lower leg inertia -->
         <inertial>
-        <origin xyz="0.0 0.00787644 -0.08928215" rpy="0 0 0" />
-        <mass value="0.03070001"/>
-        <inertia ixx="0.00012024" ixy="0.0"         ixz="0.0"
-                                   iyy="0.00012029" iyz="-0.00000305"
-                                                    izz="0.00000216"/>
+        <mass value="0.02318294"/>
+        <origin xyz="0.00000000 -0.00776716 -0.07003876" rpy="0 0 0" />
+        <inertia ixx="0.00008508" ixy="0.00000000"  ixz="0.00000000"
+                                  iyy="0.00008580"  iyz="0.00000200"
+                                                    izz="0.00000139"/>
         </inertial>
       </xacro:if>
@@ -338,5 +349,5 @@
       </contact>
     </link> <!-- END LOWER LEG LINK -->
-    <!-- KFE: Joint between the upper leg and the lower leg -->
+    <!-- KFE: Joint between the lower leg and the ankle -->
     <joint name="${prefix}_ANKLE" type="fixed">
       <parent link="${prefix}_LOWER_LEG"/>
@@ -358,9 +369,9 @@
       <!-- This link is symmetrical left or right -->
       <inertial>
-        <origin xyz="0 0 0.00035767" rpy="0 0 0" />
-        <mass value="0.00693606"/>
-        <inertia ixx="0.00000057" ixy="0.0"         ixz="0.0"
-                                   iyy="0.00000084" iyz="0.0"
-                                                    izz="0.00000053"/>
+        <origin xyz="0 0 0" rpy="0 0 0" />
+        <mass value="0.0"/>
+        <inertia ixx="0.0" ixy="0.0" ixz="0.0"
+                           iyy="0.0" iyz="0.0"
+                                     izz="0.0"/>
      </inertial>
       <!-- FOOT VISUAL -->

File: src/robot_properties_solo/resources/xacro/solo12.urdf.xacro (robot description, xacro)
@@ -13,10 +13,10 @@
     <!-- BASE LINK INERTIAL -->
     <inertial>
-        <origin xyz="0 0 0" rpy="0 0 0" />
-        <mass value="1.16115091"/>
+        <origin xyz="-0.00082966 0.00000105 -0.00060210" rpy="0 0 0" />
+        <mass value="1.25123725"/>
         <!-- The base is extremely symmetrical. -->
-        <inertia ixx="0.00578574" ixy="0.0" ixz="0.0"
-                                  iyy="0.01938108" iyz="0.0"
-                                                   izz="0.02476124"
+        <inertia ixx="0.00266220" ixy="-0.00003684" ixz="-0.00001716"
+                                  iyy="0.01388510"  iyz="-0.00000009"
+                                                    izz="0.01605370"
         />
     </inertial>
