Commit message: finalize the foot

File: src/robot_properties_solo/resources/xacro/leg.xacro (robot description, xacro)
@@ -233,8 +233,8 @@
         <geometry>
           <xacro:unless value="${is_right}">
-            <mesh filename="package://robot_properties_solo/resources/meshes/${mesh_ext}/with_foot/solo_upper_leg_left_side.${mesh_ext}"/>
-          </xacro:unless>
-          <xacro:if value="${is_right}">
-            <mesh filename="package://robot_properties_solo/resources/meshes/${mesh_ext}/with_foot/solo_upper_leg_right_side.${mesh_ext}"/>
+            <mesh filename="package://robot_properties_solo/resources/meshes/${mesh_ext}/without_foot/solo_upper_leg_left_side.${mesh_ext}"/>
+          </xacro:unless>
+          <xacro:if value="${is_right}">
+            <mesh filename="package://robot_properties_solo/resources/meshes/${mesh_ext}/without_foot/solo_upper_leg_right_side.${mesh_ext}"/>
           </xacro:if>
         </geometry>
@@ -248,8 +248,8 @@
         <geometry>
           <xacro:unless value="${is_right}">
-            <mesh filename="package://robot_properties_solo/resources/meshes/${mesh_ext}/with_foot/solo_upper_leg_left_side.${mesh_ext}"/>
-          </xacro:unless>
-          <xacro:if value="${is_right}">
-            <mesh filename="package://robot_properties_solo/resources/meshes/${mesh_ext}/with_foot/solo_upper_leg_right_side.${mesh_ext}"/>
+            <mesh filename="package://robot_properties_solo/resources/meshes/${mesh_ext}/without_foot/solo_upper_leg_left_side.${mesh_ext}"/>
+          </xacro:unless>
+          <xacro:if value="${is_right}">
+            <mesh filename="package://robot_properties_solo/resources/meshes/${mesh_ext}/without_foot/solo_upper_leg_right_side.${mesh_ext}"/>
           </xacro:if>
         </geometry>
@@ -318,8 +318,8 @@
         <geometry>
           <xacro:unless value="${is_right}">
-            <mesh filename="package://robot_properties_solo/resources/meshes/${mesh_ext}/with_foot/solo_lower_leg_left_side.${mesh_ext}"/>
-          </xacro:unless>
-          <xacro:if value="${is_right}">
-            <mesh filename="package://robot_properties_solo/resources/meshes/${mesh_ext}/with_foot/solo_lower_leg_right_side.${mesh_ext}"/>
+            <mesh filename="package://robot_properties_solo/resources/meshes/${mesh_ext}/without_foot/solo_lower_leg_v2_left_side.${mesh_ext}"/>
+          </xacro:unless>
+          <xacro:if value="${is_right}">
+            <mesh filename="package://robot_properties_solo/resources/meshes/${mesh_ext}/without_foot/solo_lower_leg_v2_right_side.${mesh_ext}"/>
           </xacro:if>
         </geometry>
@@ -333,8 +333,8 @@
         <geometry>
           <xacro:unless value="${is_right}">
-            <mesh filename="package://robot_properties_solo/resources/meshes/${mesh_ext}/with_foot/solo_lower_leg_left_side.${mesh_ext}"/>
-          </xacro:unless>
-          <xacro:if value="${is_right}">
-            <mesh filename="package://robot_properties_solo/resources/meshes/${mesh_ext}/with_foot/solo_lower_leg_right_side.${mesh_ext}"/>
+            <mesh filename="package://robot_properties_solo/resources/meshes/${mesh_ext}/without_foot/solo_lower_leg_v2_left_side.${mesh_ext}"/>
+          </xacro:unless>
+          <xacro:if value="${is_right}">
+            <mesh filename="package://robot_properties_solo/resources/meshes/${mesh_ext}/without_foot/solo_lower_leg_v2_right_side.${mesh_ext}"/>
           </xacro:if>
         </geometry>
@@ -349,5 +349,5 @@
       </contact>
     </link> <!-- END LOWER LEG LINK -->
-    <!-- KFE: Joint between the lower leg and the ankle -->
+    <!-- Joint between the lower leg and the ankle -->
     <joint name="${prefix}_ANKLE" type="fixed">
       <parent link="${prefix}_LOWER_LEG"/>
@@ -375,29 +375,4 @@
                                      izz="0.0"/>
      </inertial>
-      <!-- FOOT VISUAL -->
-      <visual>
-        <origin xyz="0 0 0" rpy="0 0 0" />
-        <geometry>
-          <mesh filename="package://robot_properties_solo/resources/meshes/${mesh_ext}/with_foot/solo_foot.${mesh_ext}"/>
-        </geometry>
-        <material name="${color_name}">
-            <color rgba="${color} ${opacity}"/>
-        </material>
-      </visual>
-      <!-- FOOT COLLISION -->
-      <collision>
-        <origin xyz="0 0 0" rpy="0 0 0" />
-        <geometry>
-            <mesh filename="package://robot_properties_solo/resources/meshes/${mesh_ext}/with_foot/solo_foot.${mesh_ext}"/>
-        </geometry>
-        <material name="${color_name}">
-            <color rgba="${color} ${opacity}"/>
-        </material>
-      </collision>
-      <!-- Bullet specific paramters -->
-      <contact>
-        <lateral_friction value="1.0"/>
-        <restitution value="0.5"/>
-      </contact>
     </link> <!-- END LOWER LEG LINK -->
   </xacro:macro>

Commit message: add some comments and make some cleaning

File: src/robot_properties_solo/resources/xacro/leg.xacro (robot description, xacro)
@@ -1,5 +1,5 @@
 <?xml version="1.0"?>
 <robot xmlns:xacro="http://playerstage.sourceforge.net/gazebo/xmlschema/#interface" name="solo">
-  <!-- See TODO: add the wiki link here -->
+  <!-- See https://github.com/open-dynamic-robot-initiative/open_robot_actuator_hardware/blob/master/mechanics/quadruped_robot_12dof_v1/README.md#quadruped-robot-12dof-v1 -->
   <!-- These are absoulte distance value, the sign are decided below -->
   <xacro:property name="base_2_HAA_x" value="${214.10 * 0.001}" />
@@ -349,5 +349,7 @@
       </contact>
     </link> <!-- END LOWER LEG LINK -->
-    <!-- Joint between the lower leg and the ankle -->
+    <!-- Joint between the lower leg and the ankle,
+         this is only a dummy joint such that we
+         can assign coordinate frames to foot-->
     <joint name="${prefix}_ANKLE" type="fixed">
       <parent link="${prefix}_LOWER_LEG"/>
@@ -360,5 +362,5 @@
         <origin xyz="0 ${-KFE_2_FOOT_y} ${-KFE_2_FOOT_z}" rpy="0 0 0" />
       </xacro:if>
-      <!-- Limits (usefull?) -->
+      <!-- Limits -->
       <limit effort="1000" lower="-10" upper="10" velocity="1000"/>
       <!-- pybullet simulation parameters -->
@@ -367,5 +369,4 @@
     <link name="${prefix}_FOOT">
       <!-- FOOT INERTIAL -->
-      <!-- This link is symmetrical left or right -->
       <inertial>
         <origin xyz="0 0 0" rpy="0 0 0" />
@@ -374,6 +375,6 @@
                            iyy="0.0" iyz="0.0"
                                      izz="0.0"/>
-     </inertial>
-    </link> <!-- END LOWER LEG LINK -->
+      </inertial>
+    </link> <!-- END FOOT LINK -->
   </xacro:macro>
 </robot>
